Commit message: Correct inertia values + formulas in macro

File: soma_mse/xacro/movebase_macro.xacro (robot description, xacro)
@@ -9,4 +9,8 @@
 	<!--  -->
 	<macro name="wheel_macro" params="parent prefix xyz">
+		<property name="mass" value="0.5" />
+		<property name="radius" value="0.2" />
+		<property name="length" value="0.1" />
+		<!--  -->
 		<joint name="${prefix}_joint" type="continuous">
 			<origin xyz="${xyz}" rpy="${radians(-90)} 0.0 0.0" />
@@ -38,10 +42,13 @@
 			<inertial>
 				<origin xyz="0.0 0.0 0.0" rpy="0.0 0.0 0.0" />
-				<mass value="0.5" />
-				<inertia ixx="0.0001" ixy="0.0" ixz="0.0" iyy="0.0001" iyz="0.0" izz="0.0001" />
+				<mass value="${mass}" />
+				<inertia ixx="${mass / 12 * (3 * radius ** 2 + length ** 2)}" ixy="0.0"
+						 ixz="0.0" iyy="${mass / 12 * (3 * radius ** 2 + length ** 2)}"
+						 iyz="0.0" izz="${mass / 2 * radius ** 2}" />
+				<!-- Old values: ixx = iyy = izz = 0.0001 -->
 			</inertial>
 			<visual>
 				<geometry>
-					<cylinder radius="0.2" length="0.1" />
+					<cylinder radius="${radius}" length="${length}" />
 				</geometry>
 				<material name="red" />
@@ -49,5 +56,5 @@
 			<collision>
 				<geometry>
-					<cylinder radius="0.2" length="0.1" />
+					<cylinder radius="${radius}" length="${length}" />
 				</geometry>
 			</collision>
@@ -66,4 +73,9 @@
 	<!--  -->
 	<macro name="body_macro" params="parent">
+		<property name="mass" value="1.0" />
+		<property name="width" value="0.6" />
+		<property name="depth" value="0.40" />
+		<property name="height" value="0.6" />
+		<!--  -->
 		<joint name="body_joint" type="fixed">
 			<parent link="${parent}" />
@@ -74,11 +86,14 @@
 			<inertial>
 				<origin xyz="0.0 0.0 0.0" rpy="0.0 0.0 0.0" />
-				<mass value="1.0" />
-				<inertia ixx="0.001" ixy="0.0" ixz="0.0" iyy="0.001" iyz="0.0" izz="0.001" />
+				<mass value="${mass}" />
+				<inertia ixx="${mass / 12 * (depth ** 2 + height ** 2)}" ixy="0.0"
+						 ixz="0.0" iyy="${mass / 12 * (width ** 2 + height ** 2)}"
+						 iyz="0.0" izz="${mass / 12 * (width ** 2 + depth ** 2)}" />
+				<!-- Old values: ixx = iyy = izz = 0.001 -->
 			</inertial>
 			<visual>
 				<origin xyz="0.0 0.0 0.0" rpy="0.0 0.0 0.0" />
 				<geometry>
-					<box size="0.6 0.40 0.6" />
+					<box size="${width} ${depth} ${height}" />
 				</geometry>
 				<material name="gray" />
@@ -87,5 +102,5 @@
 				<origin xyz="0.0 0.0 0.0" rpy="0.0 0.0 0.0" />
 				<geometry>
-					<box size="0.6 0.40 0.6" />
+					<box size="${width} ${depth} ${height}" />
 				</geometry>
 			</collision>
