Commit message: Merge soma_description & soma_mse xacro files

File: soma_description/urdf/movebase_macro.xacro (robot description, xacro)
@@ -179,5 +179,5 @@
 			<parent link="${parent}" />
 			<child link="imu_link" />
-			<origin xyz="-0.1 0 0.7" rpy="0.0 0.0 0.0" />
+			<origin xyz="0 0 1.45" rpy="0.0 0.0 0.0" />
 		</joint>
 		<!-- Link -->
@@ -216,13 +216,10 @@
 		</gazebo>
 	</macro>
-	<gazebo>
-    	<plugin name="imu_plugin" filename="libgazebo_ros_imu.so">
-      		<alwaysOn>true</alwaysOn>
-      		<bodyName>base_footprint</bodyName>
-      		<topicName>imu</topicName>
-      		<serviceName>imu_service</serviceName>
-      		<gaussianNoise>0.0</gaussianNoise>
-      		<updateRate>20.0</updateRate>
-    	</plugin>
-  	</gazebo>
+	<macro name="realsense_macro" params="parent prefix *origin">
+		<link name="camera_${prefix}_mount_link" />
+		<joint name="camera_${prefix}_mount_joint" type="fixed">
+			<parent link="${parent}" />
+			<child link="camera_${prefix}_mount_link" />
+		</joint>
+	</macro>
 </robot>

File: soma_description/urdf/movebase_vlp16.xacro (robot description, xacro)
@@ -8,11 +8,26 @@
 	<!-- Use macros -->
 	<body_macro parent="base_link" />
-	<wheel_macro prefix="left_wheel" parent="base_link" xyz="0.2 0.3 0.2" />
-	<wheel_macro prefix="right_wheel" parent="base_link" xyz="0.2 -0.3 0.2" />
-	<!--imu_macro parent="base_link" />-->
+	<wheel_macro parent="base_link" prefix="left_wheel" xyz="0.2 0.3 0.2" />
+	<wheel_macro parent="base_link" prefix="right_wheel" xyz="0.2 -0.3 0.2" />
+	<imu_macro parent="base_link" />
 	<!-- Build Velodyne -->
-	<VLP-16>
+	<VLP-16 parent="base_link" name="velodyne" topic="/velodyne_points">
 		<origin parent="base_link" xyz="0.25 0.0 0.7" rpy="0.0 0.0 0.0" />
 	</VLP-16>
+	<!-- Build Realsense -->
+	<!-- Front -->
+	<realsense_macro parent="base_link" prefix="f">
+		<origin xyz="0.85 0.1 0.61" rpy="0.0 0.0 0.0" />
+	</realsense_macro>
+	<sensor_d435 parent="camera_f_mount_link" name="camera_f">
+		<origin xyz="0.0 0.0 0.0" rpy="0.0 0.2617 0.0" />
+	</sensor_d435>
+	<!-- Rear -->
+	<realsense_macro parent="base_link" prefix="r">
+		<origin xyz="-0.2 0.0 0.35" rpy="0.0 0.0 -3.1415" />
+	</realsense_macro>
+	<sensor_d435 parent="camera_r_mount_link" name="camera_r">
+		<origin xyz="0.0 0.0 0.0" rpy="0.0 0.2617 0.0" />
+	</sensor_d435>
 	<!-- Gazebo ROS control -->
 	<gazebo>
@@ -30,4 +45,12 @@
 			</robotSimType>
 		</plugin>
-	</gazebo>
+    	<plugin name="imu_plugin" filename="libgazebo_ros_imu.so">
+      		<alwaysOn>true</alwaysOn>
+      		<bodyName>base_footprint</bodyName>
+      		<topicName>imu</topicName>
+      		<serviceName>imu_service</serviceName>
+      		<gaussianNoise>0.0</gaussianNoise>
+      		<updateRate>20.0</updateRate>
+    	</plugin>
+  	</gazebo>
 </robot>

Commit message: Correct realsense_macro + use right movebase_macro

File: soma_description/urdf/movebase_macro.xacro (robot description, xacro)
@@ -15,5 +15,6 @@
 		<property name="length" value="0.1" />
 		<!-- Joint -->
-		<joint name="${prefix}_joint" type="continuous">
+		<!--joint name="${prefix}_joint" type="continuous"-->
+		<joint name="${prefix}_joint" type="fixed">
 			<origin xyz="${xyz}" rpy="${radians(-90)} 0.0 0.0" />
 			<parent link="${parent}" />
@@ -216,10 +217,14 @@
 		</gazebo>
 	</macro>
+	<!-- END IMU macro -->
+	<!-- Realsense macro -->
 	<macro name="realsense_macro" params="parent prefix *origin">
 		<link name="camera_${prefix}_mount_link" />
 		<joint name="camera_${prefix}_mount_joint" type="fixed">
+			<insert_block name="origin" />
 			<parent link="${parent}" />
 			<child link="camera_${prefix}_mount_link" />
 		</joint>
 	</macro>
+	<!-- END Realsense macro -->
 </robot>

File: soma_description/urdf/movebase_vlp16.xacro (robot description, xacro)
@@ -2,5 +2,5 @@
 <robot xmlns:xacro="http://www.ros.org/wiki/xacro" name="dtw_robot">
 	<!-- Include files -->
-	<include filename="$(find soma_mse)/xacro/movebase_macro.xacro" />
+	<include filename="$(find soma_description)/urdf/movebase_macro.xacro" />
 	<include filename="$(find velodyne_description)/urdf/VLP-16.urdf.xacro" />
 	<include filename="$(find realsense2_description)/urdf/_d435.urdf.xacro" />

Commit message: Fix wheels display issue + add doc & clarity

File: soma_description/urdf/movebase_macro.xacro (robot description, xacro)
@@ -15,6 +15,5 @@
 		<property name="length" value="0.1" />
 		<!-- Joint -->
-		<!--joint name="${prefix}_joint" type="continuous"-->
-		<joint name="${prefix}_joint" type="fixed">
+		<joint name="${prefix}_joint" type="continuous">
 			<origin xyz="${xyz}" rpy="${radians(-90)} 0.0 0.0" />
 			<parent link="${parent}" />
