Commit message: update description and hdl graph slam

File: soma_description/urdf/soma.urdf.xacro (robot description, xacro)
@@ -3,7 +3,7 @@
 	<link name="base_link">
 		<visual>
-			<origin xyz="0.45 0.0 0.0" rpy="0.0 0.0 0.0" />
+			<origin xyz="0.5 0.0 0.225" rpy="0.0 0.0 0.0" />
 			<geometry>
-				<box size="1.4 0.9 1.2" />
+				<box size="1.45 0.9 1.3" />
 			</geometry>
 		</visual>
@@ -28,12 +28,12 @@
 		<parent link="base_link" />
 		<child link="velodyne" />
-		<origin xyz="0.5 0 1.0" rpy="0.0 0.0 0.0" />
+		<origin xyz="0.5 0 1.4" rpy="0.0 0.0 0.0" />
 	</joint>
 	<!-- realsense link (front side) -->
-	<link name="camera_f_depth_optical_frame" />
+	<link name="camera_f_link" />
 	<joint name="camera_f_joint" type="fixed">
 		<parent link="base_link" />
-		<child link="camera_f_depth_optical_frame" />
-		<origin xyz="0.85 0 0.8" rpy="0.0 0.2617 0.0" />
+		<child link="camera_f_link" />
+		<origin xyz="0.85 0 0.9" rpy="0.0 0.2617 0.0" />
 	</joint>
 </robot>

Commit message: update NUC2 (20210418)

File: soma_description/urdf/soma.urdf.xacro (robot description, xacro)
@@ -31,9 +31,9 @@
 	</joint>
 	<!-- realsense link (front side) -->
-	<link name="camera_f_depth_optical_frame" />
+	<link name="camera_f_link" />
 	<joint name="camera_f_joint" type="fixed">
 		<parent link="base_link" />
-		<child link="camera_f_depth_optical_frame" />
-		<origin xyz="0.85 0 0.8" rpy="0.0 0.2617 0.0" />
+		<child link="camera_f_link" />
+		<origin xyz="0.85 0.1 0.61" rpy="0.0 0.2617 0.0" />
 	</joint>
 </robot>

Commit message: update NUC1 (20210418)

File: soma_description/urdf/soma.urdf.xacro (robot description, xacro)
@@ -35,5 +35,5 @@
 		<parent link="base_link" />
 		<child link="camera_f_depth_optical_frame" />
-		<origin xyz="0.85 0 0.8" rpy="0.0 0.2617 0.0" />
+		<origin xyz="0.85 0.1 0.8" rpy="0.0 0.2617 0.0" />
 	</joint>
 </robot>

Commit message: add urdf xacro model of "realsense" and "vlp-16"

File: soma_description/urdf/soma.urdf.xacro (robot description, xacro)
@@ -1,4 +1,11 @@
 <?xml version="1.0"?>
 <robot xmlns:xacro="http://www.ros.org/wiki/xacro" name="soma">
+	<!--  -->
+	<!--  -->
+	<include filename="$(find realsense2_description)/urdf/_d435.urdf.xacro" />
+	<include filename="$(find velodyne_description)/urdf/VLP-16.urdf.xacro" />
+	<!--  -->
+	<!--  -->
+	<!--  -->
 	<link name="base_link">
 		<visual>
@@ -24,16 +31,26 @@
 	</joint>
 	<!-- LiDAR link (velodyne) -->
+	<!--
 	<link name="velodyne" />
 	<joint name="velodyne_joint" type="fixed">
-		<parent link="base_link" />
-		<child link="velodyne" />
+	<parent link="base_link" />
+	<child link="velodyne" />
+	<origin xyz="0.5 0 1.0" rpy="0.0 0.0 0.0" />
+	</joint>
+	-->
+	<VLP-16 parent="base_link" name="velodyne" topic="/velodyne_points">
 		<origin xyz="0.5 0 1.0" rpy="0.0 0.0 0.0" />
-	</joint>
+	</VLP-16>
 	<!-- realsense link (front side) -->
+	<!--
 	<link name="camera_f_link" />
 	<joint name="camera_f_joint" type="fixed">
-		<parent link="base_link" />
-		<child link="camera_f_link" />
+	<parent link="base_link" />
+	<child link="camera_f_link" />
+	<origin xyz="0.85 0.1 0.61" rpy="0.0 0.2617 0.0" />
+	</joint>
+	-->
+	<sensor_d435 parent="base_link" name="camera_f_link">
 		<origin xyz="0.85 0.1 0.61" rpy="0.0 0.2617 0.0" />
-	</joint>
+	</sensor_d435>
 </robot>

Commit message: fixed wheel odometry + IMU EKF filter

File: soma_description/urdf/soma.urdf.xacro (robot description, xacro)
@@ -24,8 +24,8 @@
 	</joint>
 	<!-- IMU link -->
-	<link name="imu_link" />
+	<link name="imu" />
 	<joint name="imu_joint" type="fixed">
 		<parent link="base_link" />
-		<child link="imu_link" />
+		<child link="imu" />
 		<origin xyz="0 0 1.45" rpy="0.0 0.0 0.0" />
 	</joint>

Commit message: add rear side d435

File: soma_description/urdf/soma.urdf.xacro (robot description, xacro)
@@ -54,3 +54,6 @@
 		<origin xyz="0.85 0.1 0.61" rpy="0.0 0.2617 0.0" />
 	</sensor_d435>
+	<sensor_d435 parent="base_link" name="camera_r">
+		<origin xyz="-0.2 0.0 0.35" rpy="0.0 0.2617 -3.1415" />
+	</sensor_d435>
 </robot>

Commit message: add sample for point cloud to laser scan

File: soma_description/urdf/soma.urdf.xacro (robot description, xacro)
@@ -23,4 +23,8 @@
 		<origin xyz="0.0 0.0 -0.45" rpy="0.0 0.0 0.0" />
 	</joint>
+	<!--
+	sensor links
+	D435,VLP-16,IMU, ...
+	-->
 	<!-- IMU link -->
 	<link name="imu" />
@@ -30,30 +34,27 @@
 		<origin xyz="0 0 1.45" rpy="0.0 0.0 0.0" />
 	</joint>
-	<!-- LiDAR link (velodyne) -->
-	<!--
-	<link name="velodyne" />
-	<joint name="velodyne_joint" type="fixed">
-	<parent link="base_link" />
-	<child link="velodyne" />
-	<origin xyz="0.5 0 1.0" rpy="0.0 0.0 0.0" />
-	</joint>
-	-->
+	<!-- VLP-16 -->
 	<VLP-16 parent="base_link" name="velodyne" topic="/velodyne_points">
 		<origin xyz="0.5 0 1.0" rpy="0.0 0.0 0.0" />
 	</VLP-16>
 	<!-- realsense link (front side) -->
-	<!--
-	<link name="camera_f_link" />
-	<joint name="camera_f_joint" type="fixed">
-	<parent link="base_link" />
-	<child link="camera_f_link" />
-	<origin xyz="0.85 0.1 0.61" rpy="0.0 0.2617 0.0" />
+	<link name="camera_f_mount_link" />
+	<joint name="camera_f_mount_joint" type="fixed">
+		<parent link="base_link" />
+		<child link="camera_f_mount_link" />
+		<origin xyz="0.85 0.1 0.61" rpy="0.0 0.0 0.0" />
 	</joint>
-	-->
-	<sensor_d435 parent="base_link" name="camera_f">
-		<origin xyz="0.85 0.1 0.61" rpy="0.0 0.2617 0.0" />
+	<sensor_d435 parent="camera_f_mount_link" name="camera_f">
+		<origin xyz="0.0 0.0 0.0" rpy="0.0 0.2617 0.0" />
 	</sensor_d435>
+	<!-- realsense link (rear side) -->
+	<link name="camera_r_mount_link" />
+	<joint name="camera_r_mount_joint" type="fixed">
+		<parent link="base_link" />
+		<child link="camera_r_mount_link" />
+		<origin xyz="-0.2 0.0 0.35" rpy="0.0 0.0 -3.1415" />
+	</joint>
 	<sensor_d435 parent="base_link" name="camera_r">
-		<origin xyz="-0.2 0.0 0.35" rpy="0.0 0.2617 -3.1415" />
+		<origin xyz="0.0 0.0 0.0" rpy="0.0 0.2617 0.0" />
 	</sensor_d435>
 </robot>

Commit message: Add Ackermann steering

File: soma_description/urdf/soma.urdf.xacro (robot description, xacro)
@@ -1,60 +1,50 @@
 <?xml version="1.0"?>
-<robot xmlns:xacro="http://www.ros.org/wiki/xacro" name="soma">
-	<!--  -->
-	<!--  -->
-	<include filename="$(find realsense2_description)/urdf/_d435.urdf.xacro" />
+<robot xmlns:xacro="http://www.ros.org/wiki/xacro" name="dtw_robot">
+	<!-- Include files -->
+	<include filename="$(find soma_description)/urdf/ackermann_macro.xacro" />
 	<include filename="$(find velodyne_description)/urdf/VLP-16.urdf.xacro" />
-	<!--  -->
-	<!--  -->
-	<!--  -->
-	<link name="base_link">
-		<visual>
-			<origin xyz="0.45 0.0 0.0" rpy="0.0 0.0 0.0" />
-			<geometry>
-				<box size="1.4 0.9 1.2" />
-			</geometry>
-		</visual>
-	</link>
-	<!-- Base footprint is on the ground under the robot -->
-	<link name="base_footprint" />
-	<joint name="base_footprint_joint" type="fixed">
-		<parent link="base_link" />
-		<child link="base_footprint" />
-		<origin xyz="0.0 0.0 -0.45" rpy="0.0 0.0 0.0" />
-	</joint>
-	<!--
-	sensor links
-	D435,VLP-16,IMU, ...
-	-->
-	<!-- IMU link -->
-	<link name="imu" />
-	<joint name="imu_joint" type="fixed">
-		<parent link="base_link" />
-		<child link="imu" />
-		<origin xyz="0 0 1.45" rpy="0.0 0.0 0.0" />
-	</joint>
-	<!-- VLP-16 -->
-	<VLP-16 parent="base_link" name="velodyne" topic="/velodyne_points">
-		<origin xyz="0.5 0 1.0" rpy="0.0 0.0 0.0" />
+	<include filename="$(find soma_description)/urdf/sensors_macro.xacro" />
+	<!-- Empty link to use Gazebo -->
+	<link name="base_link" />
+	<!-- Build Ackermann movebase -->
+	<ackermann_macro parent="base_link" />
+	<!-- Build Velodyne -->
+	<VLP-16 parent="body_link" name="velodyne" topic="/velodyne_points">
+		<origin parent="body_link" xyz="0.25 0.0 0.7" rpy="0.0 0.0 0.0" />
 	</VLP-16>
-	<!-- realsense link (front side) -->
-	<link name="camera_f_mount_link" />
-	<joint name="camera_f_mount_joint" type="fixed">
-		<parent link="base_link" />
-		<child link="camera_f_mount_link" />
+	<!-- Build IMU -->
+	<imu_macro parent="body_link" />
+	<!-- Build Realsense -->
+	<!-- Front -->
+	<realsense_macro parent="body_link" prefix="f">
 		<origin xyz="0.85 0.1 0.61" rpy="0.0 0.0 0.0" />
-	</joint>
-	<sensor_d435 parent="camera_f_mount_link" name="camera_f">
-		<origin xyz="0.0 0.0 0.0" rpy="0.0 0.2617 0.0" />
-	</sensor_d435>
-	<!-- realsense link (rear side) -->
-	<link name="camera_r_mount_link" />
-	<joint name="camera_r_mount_joint" type="fixed">
-		<parent link="base_link" />
-		<child link="camera_r_mount_link" />
+	</realsense_macro>
+	<!-- Rear -->
+	<realsense_macro parent="body_link" prefix="r">
 		<origin xyz="-0.2 0.0 0.35" rpy="0.0 0.0 -3.1415" />
-	</joint>
-	<sensor_d435 parent="camera_r_mount_link" name="camera_r">
-		<origin xyz="0.0 0.0 0.0" rpy="0.0 0.2617 0.0" />
-	</sensor_d435>
+	</realsense_macro>
+	<!-- Gazebo ROS control -->
+	<gazebo>
+		<plugin name="gazebo_ros_control" filename="libgazebo_ros_control.so">
+			<robotNamespace>
+				/dtw_robot
+			</robotNamespace>
+			<robotSimType>
+				gazebo_ros_control/DefaultRobotHWSim
+				<robotSimType>
+					<legacyModeNS>
+						true
+					</legacyModeNS>
+				</robotSimType>
+			</robotSimType>
+		</plugin>
+    	<plugin name="imu_plugin" filename="libgazebo_ros_imu.so">
+      		<alwaysOn>true</alwaysOn>
+      		<bodyName>base_footprint</bodyName>
+      		<topicName>imu</topicName>
+      		<serviceName>imu_service</serviceName>
+      		<gaussianNoise>0.0</gaussianNoise>
+      		<updateRate>20.0</updateRate>
+    	</plugin>
+  	</gazebo>
 </robot>

Commit message: Enable/disable sensors for debug

File: soma_description/urdf/soma.urdf.xacro (robot description, xacro)
@@ -1,29 +1,33 @@
 <?xml version="1.0"?>
 <robot xmlns:xacro="http://www.ros.org/wiki/xacro" name="soma">
+	<property name="sensors_enabled" value="false"/>
 	<!-- Include files -->
 	<include filename="$(find soma_description)/urdf/ackermann_macro.xacro" />
-	<include filename="$(find velodyne_description)/urdf/VLP-16.urdf.xacro" />
-	<include filename="$(find soma_description)/urdf/sensors_macro.xacro" />
+	<if value="${sensors_enabled}">
+		<include filename="$(find soma_description)/urdf/sensors_macro.xacro" />
+	</if>
 	<!-- Empty link to use Gazebo -->
 	<link name="base_link" />
 	<!-- Build Ackermann movebase -->
 	<ackermann_macro parent="base_link" />
-	<!-- Build IMU -->
-	<imu_macro parent="body_bottom_link">
-		<origin xyz="${-0.525 + 0.05/2} 0.0 ${1.40 - 0.25 + 0.025/2}" rpy="0.0 0.0 0.0" />
-	</imu_macro>
-	<!-- Build Realsense -->
-	<!-- Front -->
-	<realsense_macro parent="body_bottom_link" prefix="f">
-		<origin xyz="0.325 0.0 ${1.10 - 0.25}" rpy="0.0 0.0 0.0" />
-	</realsense_macro>
-	<!-- Rear -->
-	<realsense_macro parent="body_bottom_link" prefix="r">
-		<origin xyz="-0.525 0.0 ${1.10 - 0.25}" rpy="0.0 0.0 ${-pi}" />
-	</realsense_macro>
-	<!-- Build Velodyne -->
-	<velodyne_macro parent="body_bottom_link">
-		<origin xyz="0.075 0.0 ${1.70 - 0.25}" rpy="0.0 0.0 0.0" />
-	</velodyne_macro>
+	<if value="${sensors_enabled}">
+		<!-- Build IMU -->
+		<imu_macro parent="body_bottom_link">
+			<origin xyz="${-0.525 + 0.05/2} 0.0 ${1.40 - 0.25 + 0.025/2}" rpy="0.0 0.0 0.0" />
+		</imu_macro>
+		<!-- Build Realsense -->
+		<!-- Front -->
+		<realsense_macro parent="body_bottom_link" prefix="f">
+			<origin xyz="0.325 0.0 ${1.10 - 0.25}" rpy="0.0 0.0 0.0" />
+		</realsense_macro>
+		<!-- Rear -->
+		<realsense_macro parent="body_bottom_link" prefix="r">
+			<origin xyz="-0.525 0.0 ${1.10 - 0.25}" rpy="0.0 0.0 ${-pi}" />
+		</realsense_macro>
+		<!-- Build Velodyne -->
+		<velodyne_macro parent="body_bottom_link">
+			<origin xyz="0.075 0.0 ${1.70 - 0.25}" rpy="0.0 0.0 0.0" />
+		</velodyne_macro>
+	</if>
 	<!-- Gazebo plugins -->
 	<gazebo>
