Commit message: Hide virtual front steer and rear wheel

File: soma_description/urdf/front_steer_macro.xacro (robot description, xacro)
@@ -10,5 +10,6 @@
             <origin xyz="${xyz}" rpy="0 0 0" />
             <axis xyz="0 0 1" rpy="0 0 0" />
-            <limit effort="0.4" velocity="1" lower="-1" upper="1"/>
+            <!-- <limit effort="0.4" velocity="1" lower="-1" upper="1"/> -->
+            <limit effort="10" velocity="5" lower="-0.2" upper="0.2"/>
             <dynamics damping="0.1"/>
         </joint>
@@ -28,12 +29,12 @@
         <link name="${prefix}_front_steer">
             <!-- Collision part -->
-            <collision>
+            <!-- <collision>
                 <origin xyz="0 0 0.3" rpy="0 0 0" />
                 <geometry>
                     <cylinder length="0.05" radius="0.1"/>
                 </geometry>
-            </collision>
+            </collision> -->
             <!-- Visual part -->
-            <visual>
+            <!-- <visual>
                 <origin xyz="0 0 0.3" rpy="0 0 0" />
                 <geometry>
@@ -41,5 +42,5 @@
                 </geometry>
                 <material name="white"/>
-            </visual>
+            </visual> -->
             <!-- Inertial part -->
             <inertial>
@@ -59,4 +60,7 @@
             <!-- <kd value="10" /> -->
         </gazebo>
+        <gazebo reference="${prefix}_front_steer_hinge">
+            <provideFeedback>true</provideFeedback>
+        </gazebo>
     </macro>
     <!-- END front wheel macro -->

File: soma_description/urdf/front_wheel_macro.xacro (robot description, xacro)
@@ -13,5 +13,6 @@
             <origin xyz="${xyz}" rpy="0 0 0" />
             <axis xyz="0 0 1" rpy="0 0 0" />
-            <limit effort="0.4" velocity="1" lower="-1" upper="1"/>
+            <!-- <limit effort="0.4" velocity="1" lower="-1" upper="1"/> -->
+            <limit effort="10" velocity="5" lower="-0.2" upper="0.2"/>
             <dynamics damping="0.1"/>
         </joint>
@@ -22,5 +23,5 @@
             <origin xyz="0.0 0.0 0.0" rpy="${-pi/2} 0 0" />
             <axis xyz="0 0 1" rpy="0 0 0" />
-            <dynamics damping="0.1"/>
+            <!-- <dynamics damping="0.1"/> -->
         </joint>
         <!-- Transmissions -->
@@ -71,12 +72,12 @@
         <link name="${prefix}_front_wheel_assembly">
             <!-- Collision part -->
-            <collision>
+            <!-- <collision>
                 <origin xyz="0 0 0.3" rpy="0 0 0" />
                 <geometry>
                     <cylinder length="0.05" radius="0.1"/>
                 </geometry>
-            </collision>
+            </collision> -->
             <!-- Visual part -->
-            <visual>
+            <!-- <visual>
                 <origin xyz="0 0 0.3" rpy="0 0 0" />
                 <geometry>
@@ -84,5 +85,5 @@
                 </geometry>
                 <material name="white"/>
-            </visual>
+            </visual> -->
             <!-- Inertial part -->
             <inertial>

File: soma_description/urdf/rear_wheel_macro.xacro (robot description, xacro)
@@ -14,5 +14,5 @@
             <axis xyz="0 0 1" rpy="0 0 0" />
             <!--limit effort="0.4" velocity="12"/-->
-            <dynamics damping="0.1"/>
+            <!-- <dynamics damping="0.1"/> -->
         </joint>
         <!-- Transmission -->
@@ -56,6 +56,6 @@
 				Gazebo/Red
             </material>
-            <!-- <mu1 value="2.5" /> -->
-            <!-- <mu2 value="2.5" /> -->
+            <!-- <mu1 value="200" /> -->
+            <!-- <mu2 value="200" /> -->
             <!-- <kp value="1000000" /> -->
             <!-- <kd value="10" /> -->

File: soma_description/urdf/virtual_rear_wheel_macro.xacro (robot description, xacro)
@@ -45,9 +45,9 @@
             </visual> -->
             <!-- Inertial part -->
-            <!-- <inertial>
+            <inertial>
                 <origin xyz="0 0 0" rpy="0 0 0" />
                 <mass value="${mass}"/>
                 <cylinder_inertia mass="${mass}" radius="${radius}" height="${length}" />
-            </inertial> -->
+            </inertial>
         </link>
         <!-- Gazebo additional parameters -->

Commit message: Add Rviz to gazebo.laucch (for debug) + collisions

File: soma_description/urdf/front_steer_macro.xacro (robot description, xacro)
@@ -29,10 +29,10 @@
         <link name="${prefix}_front_steer">
             <!-- Collision part -->
-            <!-- <collision>
+            <collision>
                 <origin xyz="0 0 0.3" rpy="0 0 0" />
                 <geometry>
                     <cylinder length="0.05" radius="0.1"/>
                 </geometry>
-            </collision> -->
+            </collision>
             <!-- Visual part -->
             <!-- <visual>

File: soma_description/urdf/front_wheel_macro.xacro (robot description, xacro)
@@ -72,10 +72,10 @@
         <link name="${prefix}_front_wheel_assembly">
             <!-- Collision part -->
-            <!-- <collision>
+            <collision>
                 <origin xyz="0 0 0.3" rpy="0 0 0" />
                 <geometry>
                     <cylinder length="0.05" radius="0.1"/>
                 </geometry>
-            </collision> -->
+            </collision>
             <!-- Visual part -->
             <!-- <visual>

File: soma_description/urdf/virtual_rear_wheel_macro.xacro (robot description, xacro)
@@ -30,10 +30,10 @@
         <link name="${prefix}_virtual_rear_wheel">
             <!-- Collision part -->
-            <!-- <collision>
+            <collision>
                 <origin xyz="0 0 0" rpy="0 0 0" />
                 <geometry>
                     <cylinder length="${length}" radius="${radius}"/>
                 </geometry>
-            </collision> -->
+            </collision>
             <!-- Visual part -->
             <!-- <visual>

Commit message: Robot working with forest ground :)

File: soma_description/urdf/front_steer_macro.xacro (robot description, xacro)
@@ -23,5 +23,5 @@
             <actuator name="${prefix}_front_steer_motor">
                 <hardwareInterface>hardware_interface/PositionJointInterface</hardwareInterface>
-                <mechanicalReduction>10</mechanicalReduction>
+                <mechanicalReduction>1</mechanicalReduction>
             </actuator>
         </transmission>

File: soma_description/urdf/front_wheel_macro.xacro (robot description, xacro)
@@ -15,5 +15,5 @@
             <!-- <limit effort="0.4" velocity="1" lower="-1" upper="1"/> -->
             <limit effort="10" velocity="5" lower="-0.2" upper="0.2"/>
-            <dynamics damping="0.1"/>
+            <!-- <dynamics damping="0.1"/> -->
         </joint>
         <!-- Initial values: effort=0.4 velocity=12 -->
@@ -24,5 +24,5 @@
             <axis xyz="0 0 1" rpy="0 0 0" />
             <limit effort="10" velocity="5"/>
-            <dynamics damping="0.1"/>
+            <!-- <dynamics damping="0.1"/> -->
         </joint>
         <!-- Transmissions -->
@@ -34,5 +34,5 @@
             <actuator name="${prefix}_front_wheel_hinge_motor">
                 <hardwareInterface>hardware_interface/PositionJointInterface</hardwareInterface>
-                <mechanicalReduction>10</mechanicalReduction>
+                <mechanicalReduction>1</mechanicalReduction>
             </actuator>
         </transmission>
@@ -99,8 +99,8 @@
 				Gazebo/Red
             </material>
-            <!-- <mu1 value="200" /> -->
-            <!-- <mu2 value="200" /> -->
-            <kp value="1000000000" />
-            <kd value="1" />
+            <mu1 value="Inf" />
+            <mu2 value="Inf" />
+            <!-- <kp value="1000000000" />
+            <kd value="1" /> -->
         </gazebo>
         <gazebo reference="${prefix}_front_wheel_assembly">
@@ -108,8 +108,8 @@
 				Gazebo/Red
             </material>
-            <mu1 value="0.5" />
+            <!-- <mu1 value="0.5" />
             <mu2 value="0.5" />
             <kp value="1000000000" />
-            <kd value="10" />
+            <kd value="10" /> -->
         </gazebo>
     </macro>

File: soma_description/urdf/rear_wheel_macro.xacro (robot description, xacro)
@@ -14,5 +14,5 @@
             <axis xyz="0 0 1" rpy="0 0 0" />
             <limit effort="10" velocity="5"/>
-            <dynamics damping="0.1"/>
+            <!-- <dynamics damping="0.1"/> -->
         </joint>
         <!-- Transmission -->
@@ -56,8 +56,8 @@
 				Gazebo/Red
             </material>
-            <mu1 value="0.5" />
-            <mu2 value="0.5" />
-            <kp value="1000000000" />
-            <kd value="10" />
+            <mu1 value="Inf" />
+            <mu2 value="Inf" />
+            <!-- <kp value="1000000000" />
+            <kd value="10" /> -->
         </gazebo>
     </macro>
