Commit message: Change/Add wheels transmissions

File: soma_description/urdf/front_wheel_macro.xacro (robot description, xacro)
@@ -13,7 +13,8 @@
             <origin xyz="${xyz}" rpy="0 0 0" />
             <axis xyz="0 0 1" rpy="0 0 0" />
-            <limit effort="100" velocity="1" lower="-1" upper="1"/>
-            <dynamics damping="0.0" friction="0.0"/>
+            <limit effort="1000000" velocity="1000000" lower="-1" upper="1"/>
+            <dynamics damping="0.1"/>
         </joint>
+        <!-- Initial values: effort=0.4 velocity=12 -->
         <joint name="${prefix}_front_wheel_rotate" type="continuous">
             <parent link="${prefix}_front_wheel_assembly"/>
@@ -21,6 +22,5 @@
             <origin xyz="0.0 0.0 0.0" rpy="0 0 0" />
             <axis xyz="0 1 0" rpy="0 0 0" />
-            <limit effort="100" velocity="50"/>
-            <dynamics damping="0.0" friction="0.0"/>
+            <dynamics damping="0.1"/>
         </joint>
 		<!-- Transmissions -->
@@ -28,8 +28,8 @@
             <type>transmission_interface/SimpleTransmission</type>
             <joint name="${prefix}_front_wheel_hinge">
-                <hardwareInterface>EffortJointInterface</hardwareInterface>
+                <hardwareInterface>hardware_interface/PositionJointInterface</hardwareInterface>
             </joint>
             <actuator name="${prefix}_front_wheel_hinge_motor">
-                <hardwareInterface>EffortJointInterface</hardwareInterface>
+                <hardwareInterface>hardware_interface/PositionJointInterface</hardwareInterface>
                 <mechanicalReduction>10</mechanicalReduction>
             </actuator>
@@ -38,8 +38,8 @@
             <type>transmission_interface/SimpleTransmission</type>
             <joint name="${prefix}_front_wheel_rotate">
-                <hardwareInterface>EffortJointInterface</hardwareInterface>
+                <hardwareInterface>hardware_interface/VelocityJointInterface</hardwareInterface>
             </joint>
             <actuator name="${prefix}_front_wheel_rotate_motor">
-                <hardwareInterface>EffortJointInterface</hardwareInterface>
+                <hardwareInterface>hardware_interface/VelocityJointInterface</hardwareInterface>
                 <mechanicalReduction>1</mechanicalReduction>
             </actuator>
@@ -99,5 +99,5 @@
 			<mu1 value="2.5" />
 			<mu2 value="2.5" />
-			<kp value="50000" />
+			<kp value="10000000" />
 			<kd value="10" />
 		</gazebo>
@@ -108,5 +108,5 @@
 			<mu1 value="2.5" />
 			<mu2 value="2.5" />
-			<kp value="50000" />
+			<kp value="10000000" />
 			<kd value="10" />
 		</gazebo>

File: soma_description/urdf/rear_wheel_macro.xacro (robot description, xacro)
@@ -1,4 +1,4 @@
 <?xml version="1.0"?>
-<robot xmlns:xacro="http://www.ros.org/wiki/xacro" name="dtw_robot">
+<robot xmlns:xacro="http://www.ros.org/wiki/xacro" name="soma">
     <!-- Rear wheel macro -->
 	<macro name="rear_wheel_macro" params="parent prefix xyz">
@@ -13,7 +13,18 @@
             <origin xyz="${xyz}" rpy="0 0 0" />
             <axis xyz="0 1 0" rpy="0 0 0" />
-            <limit effort="100" velocity="50"/>
-            <dynamics damping="0.0" friction="0.0"/>
+            <!--limit effort="0.4" velocity="12"/-->
+            <dynamics damping="0.1"/>
         </joint>
+        <!-- Transmission -->
+        <transmission name="${prefix}_rear_wheel_rotate_trans">
+            <type>transmission_interface/SimpleTransmission</type>
+            <joint name="${prefix}_rear_wheel_rotate">
+                <hardwareInterface>hardware_interface/VelocityJointInterface</hardwareInterface>
+            </joint>
+            <actuator name="${prefix}_rear_wheel_rotate_motor">
+                <hardwareInterface>hardware_interface/VelocityJointInterface</hardwareInterface>
+                <mechanicalReduction>1</mechanicalReduction>
+            </actuator>
+        </transmission>
 		<!-- Link -->
         <link name="${prefix}_rear_wheel">
@@ -47,5 +58,5 @@
 			<mu1 value="2.5" />
 			<mu2 value="2.5" />
-			<kp value="50000" />
+			<kp value="10000000" />
 			<kd value="10" />
 		</gazebo>

Commit message: Modify parameters values

File: soma_description/urdf/front_wheel_macro.xacro (robot description, xacro)
@@ -4,5 +4,5 @@
     <macro name="front_wheel_macro" params="parent prefix xyz">
         <!-- General properties used for inertia computation -->
-        <property name="mass" value="1" />
+        <property name="mass" value="0.5" />
         <property name="radius" value="0.2286" />
         <property name="length" value="0.0889" />
@@ -14,6 +14,6 @@
             <axis xyz="0 0 1" rpy="0 0 0" />
             <!-- <limit effort="0.4" velocity="1" lower="-1" upper="1"/> -->
-            <limit effort="10" velocity="5" lower="-0.2" upper="0.2"/>
-            <!-- <dynamics damping="0.1"/> -->
+            <limit effort="10" velocity="0.1" lower="-0.2" upper="0.2"/>
+            <!-- <dynamics damping="10"/> -->
         </joint>
         <!-- Initial values: effort=0.4 velocity=12 -->
@@ -21,5 +21,5 @@
             <parent link="${prefix}_front_wheel_assembly"/>
             <child link="${prefix}_front_wheel"/>
-            <origin xyz="0.0 0.0 0.0" rpy="${-pi/2} 0 0" />
+            <origin xyz="0 0 0" rpy="${-pi/2} 0 0" />
             <axis xyz="0 0 1" rpy="0 0 0" />
             <limit effort="10" velocity="5"/>
@@ -76,5 +76,5 @@
                 <origin xyz="0 0 0.3" rpy="0 0 0" />
                 <geometry>
-                    <cylinder length="0.05" radius="0.1"/>
+                    <cylinder length="0.05" radius="0.07"/>
                 </geometry>
             </collision>
@@ -83,5 +83,5 @@
                 <origin xyz="0 0 0.3" rpy="0 0 0" />
                 <geometry>
-                    <cylinder length="0.05" radius="0.1"/>
+                    <cylinder length="0.05" radius="0.07"/>
                 </geometry>
                 <material name="white"/>
@@ -91,5 +91,5 @@
                 <origin xyz="0 0 0.3" rpy="0 0 0" />
                 <mass value="0.2"/>
-                <cylinder_inertia mass="0.2" radius="0.1" height="0.05"/>
+                <cylinder_inertia mass="0.2" radius="0.07" height="0.05"/>
             </inertial>
         </link>
@@ -108,8 +108,8 @@
 				Gazebo/Red
             </material>
-            <!-- <mu1 value="0.5" />
-            <mu2 value="0.5" />
-            <kp value="1000000000" />
-            <kd value="10" /> -->
+            <mu1 value="Inf" />
+            <mu2 value="Inf" />
+            <!-- <kp value="1000000000" /> -->
+            <!-- <kd value="10" /> -->
         </gazebo>
     </macro>

File: soma_description/urdf/rear_wheel_macro.xacro (robot description, xacro)
@@ -4,5 +4,5 @@
     <macro name="rear_wheel_macro" params="parent prefix xyz">
         <!-- General properties used for inertia computation -->
-        <property name="mass" value="1" />
+        <property name="mass" value="0.5" />
         <property name="radius" value="0.2286" />
         <property name="length" value="0.0889" />
