Commit message: Each sensor can be enabled or disabled

File: soma_description/urdf/sensors_macro.xacro (robot description, xacro)
@@ -1,91 +1,104 @@
 <?xml version="1.0"?>
 <robot xmlns:xacro="http://www.ros.org/wiki/xacro" name="soma">
+	<property name="camera_enabled" value="false"/>
+	<property name="lidar_enabled" value="true"/>
+	<property name="imu_enabled" value="false"/>
 	<!-- Include files -->
-	<include filename="$(find realsense2_description)/urdf/_d435.urdf.xacro" />
-	<include filename="$(find velodyne_description)/urdf/VLP-16.urdf.xacro" />
+	<if value="${camera_enabled}">
+		<include filename="$(find realsense2_description)/urdf/_d435.urdf.xacro" />
+	</if>
+	<if value="${lidar_enabled}">
+		<include filename="$(find velodyne_description)/urdf/VLP-16.urdf.xacro" />
+	</if>
 	<!-- IMU macro -->
-	<macro name="imu_macro" params="parent *origin">
-		<!-- General properties used for inertia computation -->
-		<property name="mass" value="0.2" />
-		<property name="width" value="0.05" />
-		<property name="depth" value="0.05" />
-		<property name="height" value="0.025" />
-		<!-- Joint -->
-		<joint name="imu_joint" type="fixed">
-			<insert_block name="origin" />
-			<parent link="${parent}" />
-			<child link="imu_link" />
-		</joint>
-		<!-- Link -->
-		<link name="imu_link">
-			<!-- Inertial part -->
-			<inertial>
-				<origin xyz="0.0 0.0 0.0" rpy="0.0 0.0 0.0" />
-				<mass value="${mass}" />
-				<!-- Inertia matrix of a parallelepiped -->
-				<inertia ixx="${mass / 12 * (depth ** 2 + height ** 2)}" ixy="0.0" ixz="0.0" iyy="${mass / 12 * (width ** 2 + height ** 2)}" iyz="0.0" izz="${mass / 12 * (width ** 2 + depth ** 2)}" />
-			</inertial>
-			<!-- Visual part -->
-			<visual>
-				<origin xyz="0.0 0.0 0.0" rpy="0.0 0.0 0.0" />
-				<geometry>
-					<box size="${width} ${depth} ${height}" />
-				</geometry>
-				<material name="red" />
-			</visual>
-			<!-- Collision part -->
-			<collision>
-				<origin xyz="0.0 0.0 0.0" rpy="0.0 0.0 0.0" />
-				<geometry>
-					<box size="${width} ${depth} ${height}" />
-				</geometry>
-			</collision>
-		</link>
-		<!-- END link -->
-		<!-- Gazebo additional parameters -->
-		<gazebo reference="imu_link">
-			<material>
-				Gazebo/Red
-			</material>
-			<gravity>true</gravity>
-			<sensor name="imu_sensor" type="imu">
-				<always_on>true</always_on>
-				<update_rate>100</update_rate>
-				<visualize>true</visualize>
-				<topic>__default_topic__</topic>
-				<plugin filename="libgazebo_ros_imu_sensor.so" name="imu_plugin">
-					<topicName>imu</topicName>
-					<bodyName>imu_link</bodyName>
-					<updateRateHZ>10.0</updateRateHZ>
-					<gaussianNoise>0.0</gaussianNoise>
-					<xyzOffset>0 0 0</xyzOffset>
-					<rpyOffset>0 0 0</rpyOffset>
-					<frameName>imu_link</frameName>
-					<initialOrientationAsReference>false</initialOrientationAsReference>
-				</plugin>
-				<pose>0 0 0 0 0 0</pose>
-			</sensor>
-		</gazebo>
-	</macro>
+	<if value="${imu_enabled}">
+		<macro name="imu_macro" params="parent *origin">
+			<!-- General properties used for inertia computation -->
+			<property name="mass" value="0.2" />
+			<property name="width" value="0.05" />
+			<property name="depth" value="0.05" />
+			<property name="height" value="0.025" />
+			<!-- Joint -->
+			<joint name="imu_joint" type="fixed">
+				<insert_block name="origin" />
+				<parent link="${parent}" />
+				<child link="imu_link" />
+			</joint>
+			<!-- Link -->
+			<link name="imu_link">
+				<!-- Inertial part -->
+				<inertial>
+					<origin xyz="0.0 0.0 0.0" rpy="0.0 0.0 0.0" />
+					<mass value="${mass}" />
+					<!-- Inertia matrix of a parallelepiped -->
+					<inertia ixx="${mass / 12 * (depth ** 2 + height ** 2)}" ixy="0.0" ixz="0.0" iyy="${mass / 12 * (width ** 2 + height ** 2)}" iyz="0.0" izz="${mass / 12 * (width ** 2 + depth ** 2)}" />
+				</inertial>
+				<!-- Visual part -->
+				<visual>
+					<origin xyz="0.0 0.0 0.0" rpy="0.0 0.0 0.0" />
+					<geometry>
+						<box size="${width} ${depth} ${height}" />
+					</geometry>
+					<material name="red" />
+				</visual>
+				<!-- Collision part -->
+				<collision>
+					<origin xyz="0.0 0.0 0.0" rpy="0.0 0.0 0.0" />
+					<geometry>
+						<box size="${width} ${depth} ${height}" />
+					</geometry>
+				</collision>
+			</link>
+			<!-- END link -->
+			<!-- Gazebo additional parameters -->
+			<gazebo reference="imu_link">
+				<material>
+					Gazebo/Red
+				</material>
+				<gravity>true</gravity>
+				<sensor name="imu_sensor" type="imu">
+					<always_on>true</always_on>
+					<update_rate>100</update_rate>
+					<visualize>true</visualize>
+					<topic>__default_topic__</topic>
+					<plugin filename="libgazebo_ros_imu_sensor.so" name="imu_plugin">
+						<topicName>imu</topicName>
+						<bodyName>imu_link</bodyName>
+						<updateRateHZ>10.0</updateRateHZ>
+						<gaussianNoise>0.0</gaussianNoise>
+						<xyzOffset>0 0 0</xyzOffset>
+						<rpyOffset>0 0 0</rpyOffset>
+						<frameName>imu_link</frameName>
+						<initialOrientationAsReference>false</initialOrientationAsReference>
+					</plugin>
+					<pose>0 0 0 0 0 0</pose>
+				</sensor>
+			</gazebo>
+		</macro>
+	</if>
 	<!-- END IMU macro -->
 	<!-- Realsense macro -->
-	<macro name="realsense_macro" params="parent prefix *origin">
-		<link name="camera_${prefix}_mount_link" />
-		<joint name="camera_${prefix}_mount_joint" type="fixed">
-			<insert_block name="origin" />
-			<parent link="${parent}" />
-			<child link="camera_${prefix}_mount_link" />
-		</joint>
-		<sensor_d435 parent="camera_${prefix}_mount_link" name="camera_${prefix}" topics_ns="camera_${prefix}">
-			<origin xyz="0.0 0.0 0.0" rpy="0.0 0.2617 0.0" />
-		</sensor_d435>
-	</macro>
+	<if value="${camera_enabled}">
+		<macro name="realsense_macro" params="parent prefix *origin">
+			<link name="camera_${prefix}_mount_link" />
+			<joint name="camera_${prefix}_mount_joint" type="fixed">
+				<insert_block name="origin" />
+				<parent link="${parent}" />
+				<child link="camera_${prefix}_mount_link" />
+			</joint>
+			<sensor_d435 parent="camera_${prefix}_mount_link" name="camera_${prefix}" topics_ns="camera_${prefix}">
+				<origin xyz="0.0 0.0 0.0" rpy="0.0 0.2617 0.0" />
+			</sensor_d435>
+		</macro>
+	</if>
 	<!-- END Realsense macro -->
 	<!-- Velodyne macro -->
-	<macro name="velodyne_macro" params="parent *origin">
-		<VLP-16 parent="${parent}" name="velodyne" topic="/velodyne_points">
-			<insert_block name="origin" />
-		</VLP-16>
-	</macro>
+	<if value="${lidar_enabled}">
+		<macro name="velodyne_macro" params="parent *origin">
+			<VLP-16 parent="${parent}" name="velodyne" topic="/velodyne_points">
+				<insert_block name="origin" />
+			</VLP-16>
+		</macro>
+	</if>
 	<!-- END Velodyne macro -->
 </robot>

File: soma_description/urdf/soma.urdf.xacro (robot description, xacro)
@@ -1,5 +1,5 @@
 <?xml version="1.0"?>
 <robot xmlns:xacro="http://www.ros.org/wiki/xacro" name="soma">
-	<property name="sensors_enabled" value="false"/>
+	<property name="sensors_enabled" value="true"/>
 	<!-- Include files -->
 	<include filename="$(find soma_description)/urdf/ackermann_macro.xacro" />
@@ -13,20 +13,28 @@
 	<if value="${sensors_enabled}">
 		<!-- Build IMU -->
-		<imu_macro parent="body_bottom_link">
-			<origin xyz="${-0.525 + 0.05/2} 0.0 ${1.40 - 0.25 + 0.025/2}" rpy="0.0 0.0 0.0" />
-		</imu_macro>
+		<if value="${imu_enabled}">
+			<imu_macro parent="body_bottom_link">
+				<origin xyz="${-0.525 + 0.05/2} 0.0 ${1.40 - 0.25 + 0.025/2}" rpy="0.0 0.0 0.0" />
+			</imu_macro>
+		</if>
 		<!-- Build Realsense -->
 		<!-- Front -->
-		<realsense_macro parent="body_bottom_link" prefix="f">
-			<origin xyz="0.325 0.0 ${1.10 - 0.25}" rpy="0.0 0.0 0.0" />
-		</realsense_macro>
+		<if value="${camera_enabled}">
+			<realsense_macro parent="body_bottom_link" prefix="f">
+				<origin xyz="0.325 0.0 ${1.10 - 0.25}" rpy="0.0 0.0 0.0" />
+			</realsense_macro>
+		</if>
 		<!-- Rear -->
-		<realsense_macro parent="body_bottom_link" prefix="r">
-			<origin xyz="-0.525 0.0 ${1.10 - 0.25}" rpy="0.0 0.0 ${-pi}" />
-		</realsense_macro>
+		<if value="${camera_enabled}">
+			<realsense_macro parent="body_bottom_link" prefix="r">
+				<origin xyz="-0.525 0.0 ${1.10 - 0.25}" rpy="0.0 0.0 ${-pi}" />
+			</realsense_macro>
+		</if>
 		<!-- Build Velodyne -->
-		<velodyne_macro parent="body_bottom_link">
-			<origin xyz="0.075 0.0 ${1.70 - 0.25}" rpy="0.0 0.0 0.0" />
-		</velodyne_macro>
+		<if value="${lidar_enabled}">
+			<velodyne_macro parent="body_bottom_link">
+				<origin xyz="0.075 0.0 ${1.70 - 0.25}" rpy="0.0 0.0 0.0" />
+			</velodyne_macro>
+		</if>
 	</if>
 	<!-- Gazebo plugins -->

Commit message: change sensor_macro name from realsense to camera

File: soma_description/urdf/sensors_macro.xacro (robot description, xacro)
@@ -81,5 +81,5 @@
 	<!-- Realsense macro -->
 	<xacro:if value="${camera_enabled}">
-		<xacro:macro name="realsense_macro" params="parent prefix *origin">
+		<xacro:macro name="camera_macro" params="parent prefix *origin">
 			<link name="camera_${prefix}_mount_link" />
 			<joint name="camera_${prefix}_mount_joint" type="fixed">

File: soma_description/urdf/soma.urdf.xacro (robot description, xacro)
@@ -21,13 +21,13 @@
 		<!-- Front -->
 		<xacro:if value="${camera_enabled}">
-			<xacro:realsense_macro parent="body_bottom_link" prefix="f">
+			<xacro:camera_macro parent="body_bottom_link" prefix="f">
 				<origin xyz="0.325 0.0 ${1.10 - 0.25}" rpy="0.0 0.0 0.0" />
-			</xacro:realsense_macro>
+			</xacro:camera_macro>
 		</xacro:if>
 		<!-- Rear -->
 		<xacro:if value="${camera_enabled}">
-			<xacro:realsense_macro parent="body_bottom_link" prefix="r">
+			<xacro:camera_macro parent="body_bottom_link" prefix="r">
 				<origin xyz="-0.525 0.0 ${1.10 - 0.25}" rpy="0.0 0.0 ${-pi}" />
-			</xacro:realsense_macro>
+			</xacro:camera_macro>
 		</xacro:if>
 		<!-- Build Velodyne -->

Commit message: Add GPS

File: soma_description/urdf/sensors_macro.xacro (robot description, xacro)
@@ -4,4 +4,5 @@
 	<property name="lidar_enabled" value="true"/>
 	<property name="imu_enabled" value="false"/>
+	<property name="gps_enabled" value="false"/>
 	<!-- Include files -->
 	<if value="${camera_enabled}">
@@ -16,7 +17,7 @@
 			<!-- General properties used for inertia computation -->
 			<property name="mass" value="0.2" />
-			<property name="width" value="0.05" />
-			<property name="depth" value="0.05" />
-			<property name="height" value="0.025" />
+			<property name="width" value="0.1" />
+			<property name="depth" value="0.1" />
+			<property name="height" value="0.1" />
 			<!-- Joint -->
 			<joint name="imu_joint" type="fixed">
@@ -59,7 +60,5 @@
 				<sensor name="imu_sensor" type="imu">
 					<always_on>true</always_on>
-					<update_rate>100</update_rate>
 					<visualize>true</visualize>
-					<topic>__default_topic__</topic>
 					<plugin filename="libgazebo_ros_imu_sensor.so" name="imu_plugin">
 						<topicName>imu</topicName>
@@ -78,4 +77,68 @@
 	</if>
 	<!-- END IMU macro -->
+	<!-- GPS macro -->
+	<if value="${gps_enabled}">
+		<macro name="gps_macro" params="parent *origin">
+			<!-- General properties used for inertia computation -->
+			<property name="mass" value="0.2" />
+			<property name="width" value="0.1" />
+			<property name="depth" value="0.1" />
+			<property name="height" value="0.1" />
+			<!-- Joint -->
+			<joint name="gps_joint" type="fixed">
+				<insert_block name="origin" />
+				<parent link="${parent}" />
+				<child link="gps_link" />
+			</joint>
+			<!-- Link -->
+			<link name="gps_link">
+				<!-- Inertial part -->
+				<inertial>
+					<origin xyz="0.0 0.0 0.0" rpy="0.0 0.0 0.0" />
+					<mass value="${mass}" />
+					<!-- Inertia matrix of a parallelepiped -->
+					<inertia ixx="${mass / 12 * (depth ** 2 + height ** 2)}" ixy="0.0" ixz="0.0" iyy="${mass / 12 * (width ** 2 + height ** 2)}" iyz="0.0" izz="${mass / 12 * (width ** 2 + depth ** 2)}" />
+				</inertial>
+				<!-- Visual part -->
+				<visual>
+					<origin xyz="0.0 0.0 0.0" rpy="0.0 0.0 0.0" />
+					<geometry>
+						<box size="${width} ${depth} ${height}" />
+					</geometry>
+					<material name="gray" />
+				</visual>
+				<!-- Collision part -->
+				<collision>
+					<origin xyz="0.0 0.0 0.0" rpy="0.0 0.0 0.0" />
+					<geometry>
+						<box size="${width} ${depth} ${height}" />
+					</geometry>
+				</collision>
+			</link>
+			<!-- END link -->
+			<!-- Gazebo additional parameters -->
+			<!-- <gazebo> -->
+			<gazebo reference="gps_link">
+				<material>
+					Gazebo/Gray
+				</material>
+				<gravity>true</gravity>
+			</gazebo>
+			<gazebo>
+				<plugin filename="libhector_gazebo_ros_gps.so" name="gps_plugin">
+					<alwaysOn>1</alwaysOn>
+					<updateRate>10.0</updateRate>
+					<bodyName>gps_link</bodyName>
+					<topicName>fix</topicName>
+					<velocityTopicName>fix_velocity</velocityTopicName>
+					<drift>5.0 5.0 5.0</drift>
+					<gaussianNoise>0.1 0.1 0.1</gaussianNoise>
+					<velocityDrift>0 0 0</velocityDrift>
+					<velocityGaussianNoise>0.1 0.1 0.1</velocityGaussianNoise>
+				</plugin>
+			</gazebo>
+		</macro>
+	</if>
+	<!-- END GPS macro -->
 	<!-- Realsense macro -->
 	<if value="${camera_enabled}">
@@ -97,5 +160,5 @@
 		<macro name="velodyne_macro" params="parent *origin">
 			<VLP-16 parent="${parent}" name="velodyne" topic="/velodyne_points" min_range="1.0" max_range="10.0" noise="0.01">
-			<!-- <VLP-16 parent="${parent}" name="velodyne" topic="/velodyne_points" min_range="1.0" max_range="10.0" noise="0.0"> -->
+				<!-- <VLP-16 parent="${parent}" name="velodyne" topic="/velodyne_points" min_range="1.0" max_range="10.0" noise="0.0"> -->
 				<!-- <VLP-16 parent="${parent}" name="velodyne" topic="/velodyne_points" min_range="0.9" max_range="130.0" noise="0.008"> -->
 				<insert_block name="origin" />

File: soma_description/urdf/soma.urdf.xacro (robot description, xacro)
@@ -15,6 +15,12 @@
 		<if value="${imu_enabled}">
 			<imu_macro parent="body_bottom_link">
-				<origin xyz="${-0.525 + 0.05/2} 0.0 ${1.40 - 0.25 + 0.025/2}" rpy="0.0 0.0 0.0" />
+				<origin xyz="${-0.525 + 0.1 + 0.1/2} 0.0 ${1.40 - 0.25 + 0.1/2}" rpy="0.0 0.0 0.0" />
 			</imu_macro>
+		</if>
+		<!-- Build GPS -->
+		<if value="${gps_enabled}">
+			<gps_macro parent="body_bottom_link">
+				<origin xyz="${-0.525 + 0.3 + 0.1/2} 0.0 ${1.40 - 0.25 + 0.1/2}" rpy="0.0 0.0 0.0" />
+			</gps_macro>
 		</if>
 		<!-- Build Realsense -->

Commit message: Add GPS

File: soma_description/urdf/sensors_macro.xacro (robot description, xacro)
@@ -1,10 +1,11 @@
 <?xml version="1.0"?>
 <robot xmlns:xacro="http://www.ros.org/wiki/xacro" name="soma">
+	<xacro:property name="imu_enabled" value="false"/>
+	<xacro:property name="gps_enabled" value="false"/>
 	<xacro:property name="camera_enabled" value="true"/>
 	<xacro:property name="lidar_enabled" value="true"/>
-	<xacro:property name="imu_enabled" value="false"/>
 	<!-- Include files -->
 	<xacro:if value="${camera_enabled}">
-	 	<xacro:include filename="$(find soma_description)/urdf/intel_realsense.urdf.xacro"/>
+		<xacro:include filename="$(find soma_description)/urdf/intel_realsense.urdf.xacro"/>
 		<!-- <xacro:include filename="$(find realsense2_description)/urdf/_d435.urdf.xacro" /> -->
 	</xacro:if>
@@ -79,4 +80,68 @@
 	</xacro:if>
 	<!-- END IMU macro -->
+	<!-- GPS macro -->
+	<if value="${gps_enabled}">
+		<macro name="gps_macro" params="parent *origin">
+			<!-- General properties used for inertia computation -->
+			<property name="mass" value="0.2" />
+			<property name="width" value="0.1" />
+			<property name="depth" value="0.1" />
+			<property name="height" value="0.1" />
+			<!-- Joint -->
+			<joint name="gps_joint" type="fixed">
+				<insert_block name="origin" />
+				<parent link="${parent}" />
+				<child link="gps_link" />
+			</joint>
+			<!-- Link -->
+			<link name="gps_link">
+				<!-- Inertial part -->
+				<inertial>
+					<origin xyz="0.0 0.0 0.0" rpy="0.0 0.0 0.0" />
+					<mass value="${mass}" />
+					<!-- Inertia matrix of a parallelepiped -->
+					<inertia ixx="${mass / 12 * (depth ** 2 + height ** 2)}" ixy="0.0" ixz="0.0" iyy="${mass / 12 * (width ** 2 + height ** 2)}" iyz="0.0" izz="${mass / 12 * (width ** 2 + depth ** 2)}" />
+				</inertial>
+				<!-- Visual part -->
+				<visual>
+					<origin xyz="0.0 0.0 0.0" rpy="0.0 0.0 0.0" />
+					<geometry>
+						<box size="${width} ${depth} ${height}" />
+					</geometry>
+					<material name="gray" />
+				</visual>
+				<!-- Collision part -->
+				<collision>
+					<origin xyz="0.0 0.0 0.0" rpy="0.0 0.0 0.0" />
+					<geometry>
+						<box size="${width} ${depth} ${height}" />
+					</geometry>
+				</collision>
+			</link>
+			<!-- END link -->
+			<!-- Gazebo additional parameters -->
+			<!-- <gazebo> -->
+			<gazebo reference="gps_link">
+				<material>
+					Gazebo/Gray
+				</material>
+				<gravity>true</gravity>
+			</gazebo>
+			<gazebo>
+				<plugin filename="libhector_gazebo_ros_gps.so" name="gps_plugin">
+					<alwaysOn>1</alwaysOn>
+					<updateRate>10.0</updateRate>
+					<bodyName>gps_link</bodyName>
+					<topicName>fix</topicName>
+					<velocityTopicName>fix_velocity</velocityTopicName>
+					<drift>5.0 5.0 5.0</drift>
+					<gaussianNoise>0.1 0.1 0.1</gaussianNoise>
+					<velocityDrift>0 0 0</velocityDrift>
+					<velocityGaussianNoise>0.1 0.1 0.1</velocityGaussianNoise>
+				</plugin>
+			</gazebo>
+		</macro>
+	</if>
+	<!-- END GPS macro -->
 	<!-- Realsense macro -->
 	<xacro:if value="${camera_enabled}">
@@ -88,5 +153,5 @@
 				<child link="camera_${prefix}_mount_link" />
 			</joint>
-			<!-- <xacro:sensor_d435 parent="camera_${prefix}_mount_link" name="camera_${prefix}" >
+			<!-- <xacro:sensor_d435 parent="camera_${prefix}_mount_link" name="camera_${prefix}">
 				<origin xyz="0.0 0.0 0.0" rpy="0.0 0.2617 0.0" />
 			</xacro:sensor_d435> -->
@@ -99,5 +164,5 @@
 		<xacro:macro name="velodyne_macro" params="parent *origin">
 			<!-- <xacro:VLP-16 parent="${parent}" name="velodyne" topic="/velodyne_points" min_range="0.0" max_range="5.0" noise="0.0"> -->
-				<xacro:VLP-16 parent="${parent}" name="velodyne" topic="/velodyne_points" min_range="0.9" max_range="130.0" noise="0.008">
+			<xacro:VLP-16 parent="${parent}" name="velodyne" topic="/velodyne_points" min_range="0.9" max_range="130.0" noise="0.008">
 				<xacro:insert_block name="origin" />
 			</xacro:VLP-16>

File: soma_description/urdf/soma.urdf.xacro (robot description, xacro)
@@ -18,4 +18,10 @@
 			</xacro:imu_macro>
 		</xacro:if>
+		<!-- Build GPS -->
+		<if value="${gps_enabled}">
+			<gps_macro parent="body_bottom_link">
+				<origin xyz="${-0.525 + 0.3 + 0.1/2} 0.0 ${1.40 - 0.25 + 0.1/2}" rpy="0.0 0.0 0.0" />
+			</gps_macro>
+		</if>
 		<!-- Build Realsense -->
 		<!-- Front -->

Commit message: fix for beach clean 220429

File: soma_description/urdf/sensors_macro.xacro (robot description, xacro)
@@ -6,5 +6,6 @@
 	<!-- Include files -->
 	<xacro:if value="${camera_enabled}">
-	 	<xacro:include filename="$(find soma_description)/urdf/intel_realsense.urdf.xacro"/>
+		<xacro:include filename="$(find soma_description)/urdf/intel_realsense.urdf.xacro"/>
+		<xacro:include filename="$(find azure_kinect_ros_driver)/urdf/azure_kinect.urdf.xacro"/>
 		<!-- <xacro:include filename="$(find realsense2_description)/urdf/_d435.urdf.xacro" /> -->
 	</xacro:if>
@@ -88,5 +89,5 @@
 				<child link="camera_${prefix}_mount_link" />
 			</joint>
-			<!-- <xacro:sensor_d435 parent="camera_${prefix}_mount_link" name="camera_${prefix}" >
+			<!-- <xacro:sensor_d435 parent="camera_${prefix}_mount_link" name="camera_${prefix}">
 				<origin xyz="0.0 0.0 0.0" rpy="0.0 0.2617 0.0" />
 			</xacro:sensor_d435> -->
@@ -95,9 +96,21 @@
 	</xacro:if>
 	<!-- END Realsense macro -->
+	<!-- Azure macro -->
+	<xacro:if value="${camera_enabled}">
+		<xacro:macro name="azure_macro" params="parent prefix *origin">
+			<!-- <link name="azure_base" /> -->
+			<joint name="soma_azure_joint" type="fixed">
+				<xacro:insert_block name="origin" />
+				<parent link="${parent}" />
+				<child link="camera_base" />
+			</joint>
+		</xacro:macro>
+	</xacro:if>
+	<!-- END Azure macro -->
 	<!-- Velodyne macro -->
 	<xacro:if value="${lidar_enabled}">
 		<xacro:macro name="velodyne_macro" params="parent *origin">
 			<!-- <xacro:VLP-16 parent="${parent}" name="velodyne" topic="/velodyne_points" min_range="0.0" max_range="5.0" noise="0.0"> -->
-				<xacro:VLP-16 parent="${parent}" name="velodyne" topic="/velodyne_points" min_range="0.9" max_range="130.0" noise="0.008">
+			<xacro:VLP-16 parent="${parent}" name="velodyne" topic="/velodyne_points" min_range="0.9" max_range="130.0" noise="0.008">
 				<xacro:insert_block name="origin" />
 			</xacro:VLP-16>

File: soma_description/urdf/soma.urdf.xacro (robot description, xacro)
@@ -31,4 +31,10 @@
 			</xacro:camera_macro>
 		</xacro:if>
+		<!-- Build Realsense -->
+		<xacro:if value="${camera_enabled}">
+			<xacro:azure_macro parent="body_bottom_link" prefix="f">
+				<origin xyz="0.325 0.0 ${1.10 - 0.25}" rpy="0.0 0.0 0.0" />
+			</xacro:azure_macro>
+		</xacro:if>
 		<!-- Build Velodyne -->
 		<xacro:if value="${lidar_enabled}">

Commit message: add ekf functions

File: soma_description/urdf/sensors_macro.xacro (robot description, xacro)
@@ -3,5 +3,5 @@
 	<xacro:property name="camera_enabled" value="true"/>
 	<xacro:property name="lidar_enabled" value="true"/>
-	<xacro:property name="imu_enabled" value="false"/>
+	<xacro:property name="imu_enabled" value="true"/>
 	<!-- Include files -->
 	<xacro:if value="${camera_enabled}">
@@ -25,8 +25,8 @@
 				<xacro:insert_block name="origin" />
 				<parent link="${parent}" />
-				<child link="imu_link" />
+				<child link="imu" />
 			</joint>
 			<!-- Link -->
-			<link name="imu_link">
+			<link name="imu">
 				<!-- Inertial part -->
 				<inertial>
@@ -54,5 +54,5 @@
 			<!-- END link -->
 			<!-- Gazebo additional parameters -->
-			<gazebo reference="imu_link">
+			<!-- <gazebo reference="imu_link">
 				<material>
 					Gazebo/Red
@@ -76,5 +76,5 @@
 					<pose>0 0 0 0 0 0</pose>
 				</sensor>
-			</gazebo>
+			</gazebo> -->
 		</xacro:macro>
 	</xacro:if>
