Commit message: Update measurements

File: soma_description/urdf/ackermann_macro.xacro (robot description, xacro)
@@ -10,22 +10,22 @@
 	<macro name="ackermann_macro" params="parent">
 		<!-- General properties used for inertia computation -->
-		<property name="mass" value="1.0" />
-		<property name="width" value="0.6" />
-		<property name="depth" value="0.40" />
-		<property name="height" value="0.6" />
-		<!-- Body joint -->
-		<joint name="body_joint" type="fixed">
+		<property name="mass" value="250" />
+		<property name="width" value="1.05" />
+		<property name="depth" value="0.70" />
+		<property name="height" value="1.7" />
+		<!-- Bottom body joint -->
+		<joint name="body_bottom_joint" type="fixed">
 			<parent link="${parent}" />
-			<child link="body_link" />
-			<origin xyz="0 0 0.4" rpy="0.0 0.0 0.0" />
+			<child link="body_bottom_link" />
+			<origin xyz="0 0 ${0.2286 + 0.5/2}" rpy="0.0 0.0 0.0" />
 		</joint>
-		<!-- Body link -->
-		<link name="body_link">
+		<!-- Bottom body link -->
+		<link name="body_bottom_link">
 			<!-- Inertial part -->
 			<inertial>
 				<origin xyz="0.0 0.0 0.0" rpy="0.0 0.0 0.0" />
-				<mass value="${mass}" />
+				<mass value="${0.8*mass}" />
 				<!-- Inertia matrix of a parallelepiped -->
-                <parallelepiped_inertia mass="${mass}" width="${width}" height="${height}" depth="${depth}" />
+                <parallelepiped_inertia mass="${mass}" width="${width}" height="0.5" depth="${depth}" />
 				<!-- Old values: ixx = iyy = izz = 0.001 -->
 			</inertial>
@@ -34,5 +34,5 @@
 				<origin xyz="0.0 0.0 0.0" rpy="0.0 0.0 0.0" />
 				<geometry>
-					<box size="${width} ${depth} ${height}" />
+					<box size="${width} ${depth} 0.5" />
 				</geometry>
 				<material name="gray" />
@@ -42,11 +42,89 @@
 				<origin xyz="0.0 0.0 0.0" rpy="0.0 0.0 0.0" />
 				<geometry>
-					<box size="${width} ${depth} ${height}" />
+					<box size="${width} ${depth} 0.5" />
 				</geometry>
 			</collision>
 		</link>
-		<!-- END link -->
+		<!-- END bottom body link -->
 		<!-- Gazebo additional parameters -->
-		<gazebo reference="body_link">
+		<gazebo reference="body_bottom_link">
+			<material>
+				Gazebo/Gray
+			</material>
+		</gazebo>
+		<!-- Middle body joint -->
+		<joint name="body_middle_joint" type="fixed">
+			<parent link="${parent}" />
+			<child link="body_middle_link" />
+			<origin xyz="-0.1 0 ${0.2286 + 0.5 + 0.9/2}" rpy="0.0 0.0 0.0" />
+		</joint>
+		<!-- Middle body link -->
+		<link name="body_middle_link">
+			<!-- Inertial part -->
+			<inertial>
+				<origin xyz="0.0 0.0 0.0" rpy="0.0 0.0 0.0" />
+				<mass value="${0.19*mass}" />
+				<!-- Inertia matrix of a parallelepiped -->
+                <parallelepiped_inertia mass="${mass}" width="0.85" height="0.9" depth="${depth}" />
+				<!-- Old values: ixx = iyy = izz = 0.001 -->
+			</inertial>
+			<!-- Visual part -->
+			<visual>
+				<origin xyz="0.0 0.0 0.0" rpy="0.0 0.0 0.0" />
+				<geometry>
+					<box size="0.85 ${depth} 0.9" />
+				</geometry>
+				<material name="gray" />
+			</visual>
+			<!-- Collision part -->
+			<collision>
+				<origin xyz="0.0 0.0 0.0" rpy="0.0 0.0 0.0" />
+				<geometry>
+					<box size="0.85 ${depth} 0.9" />
+				</geometry>
+			</collision>
+		</link>
+		<!-- END middle body link -->
+		<!-- Gazebo additional parameters -->
+		<gazebo reference="body_middle_link">
+			<material>
+				Gazebo/Gray
+			</material>
+		</gazebo>
+		<!-- Top body joint -->
+		<joint name="body_top_joint" type="fixed">
+			<parent link="${parent}" />
+			<child link="body_top_link" />
+			<origin xyz="0.075 0 ${0.2286 + 0.5 + 0.9 + 0.3/2}" rpy="0.0 0.0 0.0" />
+		</joint>
+		<!-- Top body link -->
+		<link name="body_top_link">
+			<!-- Inertial part -->
+			<inertial>
+				<origin xyz="0.0 0.0 0.0" rpy="0.0 0.0 0.0" />
+				<mass value="${0.01*mass}" />
+				<!-- Inertia matrix of a parallelepiped -->
+                <parallelepiped_inertia mass="${mass}" width="0.05" height="0.3" depth="0.05" />
+				<!-- Old values: ixx = iyy = izz = 0.001 -->
+			</inertial>
+			<!-- Visual part -->
+			<visual>
+				<origin xyz="0.0 0.0 0.0" rpy="0.0 0.0 0.0" />
+				<geometry>
+					<box size="0.05 0.05 0.3" />
+				</geometry>
+				<material name="gray" />
+			</visual>
+			<!-- Collision part -->
+			<collision>
+				<origin xyz="0.0 0.0 0.0" rpy="0.0 0.0 0.0" />
+				<geometry>
+					<box size="0.05 0.05 0.3" />
+				</geometry>
+			</collision>
+		</link>
+		<!-- END top body link -->
+		<!-- Gazebo additional parameters -->
+		<gazebo reference="body_top_link">
 			<material>
 				Gazebo/Gray
@@ -54,8 +132,8 @@
 		</gazebo>
         <!-- Build wheels -->
-        <front_wheel_macro parent="body_link" prefix="left" xyz="0.2 0.3 -0.2" />
-        <front_wheel_macro parent="body_link" prefix="right" xyz="0.2 -0.3 -0.2" />
-        <rear_wheel_macro parent="body_link" prefix="left" xyz="-0.2 0.3 -0.2" />
-        <rear_wheel_macro parent="body_link" prefix="right" xyz="-0.2 -0.3 -0.2" />
+        <front_wheel_macro parent="body_bottom_link" prefix="left" xyz="${width/2} ${depth/2 + 0.0889} ${-0.5/2}" />
+        <front_wheel_macro parent="body_bottom_link" prefix="right" xyz="${width/2} ${-depth/2 - 0.0889} ${-0.5/2}" />
+        <rear_wheel_macro parent="body_bottom_link" prefix="left" xyz="${-width/2} ${depth/2 + 0.0889} ${-0.5/2}" />
+        <rear_wheel_macro parent="body_bottom_link" prefix="right" xyz="${-width/2} ${-depth/2 - 0.0889} ${-0.5/2}" />
     </macro>
 </robot>

File: soma_description/urdf/front_wheel_macro.xacro (robot description, xacro)
@@ -4,7 +4,7 @@
 	<macro name="front_wheel_macro" params="parent prefix xyz">
 		<!-- General properties used for inertia computation -->
-		<property name="mass" value="0.5" />
-		<property name="radius" value="0.2" />
-		<property name="length" value="0.1" />
+		<property name="mass" value="12" />
+		<property name="radius" value="0.2286" />
+		<property name="length" value="0.0889" />
 		<!-- Joints -->
         <joint name="${prefix}_front_wheel_hinge" type="revolute">
@@ -32,5 +32,5 @@
             <actuator name="${prefix}_front_wheel_hinge_motor">
                 <hardwareInterface>EffortJointInterface</hardwareInterface>
-                <mechanicalReduction>1</mechanicalReduction>
+                <mechanicalReduction>10</mechanicalReduction>
             </actuator>
         </transmission>

File: soma_description/urdf/rear_wheel_macro.xacro (robot description, xacro)
@@ -4,7 +4,7 @@
 	<macro name="rear_wheel_macro" params="parent prefix xyz">
 		<!-- General properties used for inertia computation -->
-		<property name="mass" value="0.5" />
-		<property name="radius" value="0.2" />
-		<property name="length" value="0.1" />
+		<property name="mass" value="12" />
+		<property name="radius" value="0.2286" />
+		<property name="length" value="0.0889" />
 		<!-- Joint -->
         <joint name="${prefix}_rear_wheel_rotate" type="continuous">

File: soma_description/urdf/sensors_macro.xacro (robot description, xacro)
@@ -4,7 +4,7 @@
 	<include filename="$(find realsense2_description)/urdf/_d435.urdf.xacro" />
 	<!-- IMU macro -->
-	<macro name="imu_macro" params="parent">
+	<macro name="imu_macro" params="parent *origin">
 		<!-- General properties used for inertia computation -->
-		<property name="mass" value="0.5" />
+		<property name="mass" value="0.2" />
 		<property name="width" value="0.05" />
 		<property name="depth" value="0.05" />
@@ -12,7 +12,7 @@
 		<!-- Joint -->
 		<joint name="imu_joint" type="fixed">
+			<insert_block name="origin" />
 			<parent link="${parent}" />
 			<child link="imu_link" />
-			<origin xyz="0 0 1.45" rpy="0.0 0.0 0.0" />
 		</joint>
 		<!-- Link -->

File: soma_description/urdf/soma.urdf.xacro (robot description, xacro)
@@ -10,17 +10,19 @@
 	<ackermann_macro parent="base_link" />
 	<!-- Build Velodyne -->
-	<VLP-16 parent="body_link" name="velodyne" topic="/velodyne_points">
-		<origin parent="body_link" xyz="0.25 0.0 0.7" rpy="0.0 0.0 0.0" />
+	<VLP-16 parent="body_bottom_link" name="velodyne" topic="/velodyne_points">
+		<origin xyz="0.075 0.0 ${1.70 - 0.25}" rpy="0.0 0.0 0.0" />
 	</VLP-16>
 	<!-- Build IMU -->
-	<imu_macro parent="body_link" />
+	<imu_macro parent="body_bottom_link">
+		<origin xyz="${-0.525 + 0.05/2} 0.0 ${1.40 - 0.25 + 0.025/2}" rpy="0.0 0.0 0.0" />
+	</imu_macro>
 	<!-- Build Realsense -->
 	<!-- Front -->
-	<realsense_macro parent="body_link" prefix="f">
-		<origin xyz="0.85 0.1 0.61" rpy="0.0 0.0 0.0" />
+	<realsense_macro parent="body_bottom_link" prefix="f">
+		<origin xyz="0.325 0.0 ${1.10 - 0.25}" rpy="0.0 0.0 0.0" />
 	</realsense_macro>
 	<!-- Rear -->
-	<realsense_macro parent="body_link" prefix="r">
-		<origin xyz="-0.2 0.0 0.35" rpy="0.0 0.0 -3.1415" />
+	<realsense_macro parent="body_bottom_link" prefix="r">
+		<origin xyz="-0.525 0.0 ${1.10 - 0.25}" rpy="0.0 0.0 ${-pi}" />
 	</realsense_macro>
 	<!-- Gazebo ROS control -->

Commit message: Ackermann test working

File: soma_description/urdf/ackermann_macro.xacro (robot description, xacro)
@@ -7,5 +7,4 @@
     <include filename="$(find soma_description)/urdf/front_wheel_macro.xacro" />
     <include filename="$(find soma_description)/urdf/rear_wheel_macro.xacro" />
-	<include filename="$(find soma_description)/urdf/ackermann_steer_macro.xacro" />
 	<!-- Ackermann macro -->
 	<macro name="ackermann_macro" params="parent">
@@ -133,11 +132,11 @@
 		</gazebo>
 		<!-- Build links and joints for ackermann_steering_controller -->
-		<!--ackermann_steer_macro parent="body_bottom_link" xyz="${width/2} 0 ${0.5 + 0.2/2}" /-->
+		<!--front_wheel_macro parent="body_bottom_link" prefix="ackermann" xyz="${width/2 + 0.5} 0 ${-0.5/2}" /-->
 		<!--rear_wheel_macro parent="body_bottom_link" prefix="ackermann" xyz="${-width/2 - 0.5} 0 ${-0.5/2}" /-->
         <!-- Build wheels -->
-        <front_wheel_macro parent="body_bottom_link" prefix="left" xyz="${width/2} ${depth/2 + 0.0889} ${-0.5/2}" />
-        <front_wheel_macro parent="body_bottom_link" prefix="right" xyz="${width/2} ${-depth/2 - 0.0889} ${-0.5/2}" />
-        <rear_wheel_macro parent="body_bottom_link" prefix="left" xyz="${-width/2} ${depth/2 + 0.0889} ${-0.5/2}" />
-        <rear_wheel_macro parent="body_bottom_link" prefix="right" xyz="${-width/2} ${-depth/2 - 0.0889} ${-0.5/2}" />
+        <front_wheel_macro parent="body_bottom_link" prefix="left" xyz="${width/2} ${depth/2 + 0.0889} -0.2" />
+        <front_wheel_macro parent="body_bottom_link" prefix="right" xyz="${width/2} ${-depth/2 - 0.0889} -0.2" />
+        <rear_wheel_macro parent="body_bottom_link" prefix="left" xyz="${-width/2} ${depth/2 + 0.0889} -0.2" />
+        <rear_wheel_macro parent="body_bottom_link" prefix="right" xyz="${-width/2} ${-depth/2 - 0.0889} -0.2" />
     </macro>
 </robot>

File: soma_description/urdf/front_wheel_macro.xacro (robot description, xacro)
@@ -13,5 +13,5 @@
             <origin xyz="${xyz}" rpy="0 0 0" />
             <axis xyz="0 0 1" rpy="0 0 0" />
-            <limit effort="1000000" velocity="1000000" lower="-1" upper="1"/>
+            <limit effort="0.4" velocity="1" lower="-1" upper="1"/>
             <dynamics damping="0.1"/>
         </joint>
@@ -97,7 +97,7 @@
 				Gazebo/Red
 			</material>
-			<mu1 value="2.5" />
-			<mu2 value="2.5" />
-			<kp value="10000000" />
+			<mu1 value="200" />
+			<mu2 value="200" />
+			<kp value="1000000" />
 			<kd value="10" />
 		</gazebo>
@@ -106,7 +106,7 @@
 				Gazebo/Red
 			</material>
-			<mu1 value="2.5" />
-			<mu2 value="2.5" />
-			<kp value="10000000" />
+			<mu1 value="200" />
+			<mu2 value="200" />
+			<kp value="1000000" />
 			<kd value="10" />
 		</gazebo>

File: soma_description/urdf/rear_wheel_macro.xacro (robot description, xacro)
@@ -58,5 +58,5 @@
 			<mu1 value="2.5" />
 			<mu2 value="2.5" />
-			<kp value="10000000" />
+			<kp value="1000000" />
 			<kd value="10" />
 		</gazebo>

File: soma_description/urdf/test.urdf.xacro (robot description, xacro)
@@ -8,5 +8,5 @@
 	    <parent link="base_link" />
 		<child link="body_link" />
-			<origin xyz="0 0 0.5" rpy="0.0 0.0 0.0" />
+			<origin xyz="0 0 0" rpy="0.0 0.0 0.0" />
     </joint>
     <!-- Bottom body link -->
@@ -15,7 +15,8 @@
         <inertial>
             <origin xyz="0.0 0.0 0.0" rpy="0.0 0.0 0.0" />
-            <mass value="10" />
+            <mass value="5" />
             <!-- Inertia matrix of a parallelepiped -->
-            <parallelepiped_inertia mass="10" width="1.6" depth="0.3" height="0.2" />
+            <!--parallelepiped_inertia mass="5" width="0.5" depth="0.12" height="0.1" /-->
+            <inertia ixx="0.001" iyy="0.001" izz="0.001" ixy="0" ixz="0" iyz="0" />
             <!-- Old values: ixx = iyy = izz = 0.001 -->
         </inertial>
@@ -24,5 +25,5 @@
             <origin xyz="0.0 0.0 0.0" rpy="0.0 0.0 0.0" />
             <geometry>
-                <box size="1.6 0.3 0.2" />
+                <box size="0.5 0.12 0.1" />
             </geometry>
             <material name="red" />
@@ -32,5 +33,5 @@
             <origin xyz="0.0 0.0 0.0" rpy="0.0 0.0 0.0" />
             <geometry>
-                <box size="1.6 0.3 0.2" />
+                <box size="0.5 0.12 0.1" />
             </geometry>
         </collision>
@@ -47,8 +48,8 @@
         <parent link="body_link"/>
         <child link="front_wheel_assembly"/>
-        <origin xyz="0.7 0 -0.3" rpy="0 0 0" />
+        <origin xyz="${0.5/2-0.05} 0 ${0.1+0.02}" rpy="0 0 0" />
         <axis xyz="0 0 1" rpy="0 0 0" />
-        <limit effort="0.4" velocity="12" lower="-1" upper="1"/>
-        <dynamics damping="0.1"/>
+        <limit effort="10" velocity="5" lower="${-pi/2}" upper="${pi/2}"/>
+        <!--dynamics damping="0.1"/-->
     </joint>
     <!-- Initial values: effort=0.4 velocity=12 -->
@@ -56,7 +57,7 @@
         <parent link="front_wheel_assembly"/>
         <child link="front_wheel"/>
-        <origin xyz="0 0 0" rpy="0 0 0" />
-        <axis xyz="0 1 0" rpy="0 0 0" />
-        <dynamics damping="0.1"/>
+        <origin xyz="0 0 ${-0.1-0.02}" rpy="${-pi/2} 0 0" />
+        <axis xyz="0 0 1" rpy="0 0 0" />
+        <!--dynamics damping="0.1"/-->
     </joint>
     <!-- Transmissions -->
@@ -68,31 +69,21 @@
         <actuator name="front_wheel_hinge_motor">
             <hardwareInterface>hardware_interface/PositionJointInterface</hardwareInterface>
-            <mechanicalReduction>10</mechanicalReduction>
+            <mechanicalReduction>1</mechanicalReduction>
         </actuator>
     </transmission>
-    <transmission name="front_wheel_rotate_trans">
-        <type>transmission_interface/SimpleTransmission</type>
-        <joint name="front_wheel_rotate">
-            <hardwareInterface>hardware_interface/VelocityJointInterface</hardwareInterface>
-        </joint>
-        <actuator name="front_wheel_rotate_motor">
-            <hardwareInterface>hardware_interface/VelocityJointInterface</hardwareInterface>
-            <mechanicalReduction>1</mechanicalReduction>
-        </actuator>
-    </transmission>
     <!-- Links -->
     <link name="front_wheel">
         <!-- Collision part -->
         <collision>
-            <origin xyz="0 0 0" rpy="0 ${pi/2} ${pi/2}" />
-            <geometry>
-                <cylinder length="0.1" radius="0.2"/>
+            <origin xyz="0 0 0" rpy="0 0 0" />
+            <geometry>
+                <cylinder length="0.1" radius="0.1"/>
             </geometry>
         </collision>
         <!-- Visual part -->
         <visual>
-            <origin xyz="0 0 0" rpy="0 ${pi/2} ${pi/2}" />
-            <geometry>
-                <cylinder length="0.1" radius="0.2"/>
+            <origin xyz="0 0 0" rpy="0 0 0" />
+            <geometry>
+                <cylinder length="0.1" radius="0.1"/>
             </geometry>
             <material name="black"/>
@@ -100,7 +91,8 @@
         <!-- Inertial part -->
         <inertial>
-            <origin xyz="0 0 0" rpy="0 ${pi/2} ${pi/2}" />
-            <mass value="1"/>
-            <cylinder_inertia mass="1" radius="0.2" height="0.1" />
+            <origin xyz="0 0 0" rpy="0 0 0" />
+            <mass value="1"/>
+            <inertia ixx="0.001" iyy="0.001" izz="0.001" ixy="0" ixz="0" iyz="0" />
+            <!--cylinder_inertia mass="1" radius="0.1" height="0.1" /-->
         </inertial>
     </link>
@@ -108,14 +100,14 @@
         <!-- Collision part -->
         <collision>
-            <origin xyz="0 0 0" rpy="0 ${pi/2} ${pi/2}" />
-            <geometry>
-                <cylinder length="0.05" radius="0.1"/>
+            <origin xyz="0 0 0" rpy="0 0 0" />
+            <geometry>
+                <cylinder length="0.02" radius="0.05"/>
             </geometry>
         </collision>
         <!-- Visual part -->
         <visual>
-            <origin xyz="0 0 0" rpy="0 ${pi/2} ${pi/2}" />
-            <geometry>
-                <cylinder length="0.05" radius="0.1"/>
+            <origin xyz="0 0 0" rpy="0 0 0" />
+            <geometry>
+                <cylinder length="0.02" radius="0.05"/>
             </geometry>
             <material name="white"/>
@@ -123,7 +115,8 @@
         <!-- Inertial part -->
         <inertial>
-            <origin xyz="0 0 0" rpy="0 ${pi/2} ${pi/2}" />
-            <mass value="0.2"/>
-            <cylinder_inertia mass="0.2" radius="0.1" height="0.5"/>
+            <origin xyz="0 0 0" rpy="0 0 0" />
+            <mass value="1"/>
+            <inertia ixx="0.001" iyy="0.001" izz="0.001" ixy="0" ixz="0" iyz="0" />
+            <!--cylinder_inertia mass="1" radius="0.05" height="0.02"/-->
         </inertial>
     </link>
@@ -133,8 +126,11 @@
             Gazebo/Red
         </material>
-        <mu1 value="2.5" />
-        <mu2 value="2.5" />
-        <kp value="10000000" />
-        <kd value="10" />
+        <!--mu1 value="2.5" /-->
+        <!--mu2 value="2.5" /-->
+        <!--kp value="1000000" /-->
+        <!--kd value="10" /-->
+    </gazebo>
+    <gazebo reference="front_wheel_rotate">
+        <provideFeedback>true</provideFeedback>
     </gazebo>
     <gazebo reference="front_wheel_assembly">
@@ -142,8 +138,8 @@
             Gazebo/Red
         </material>
-        <mu1 value="2.5" />
-        <mu2 value="2.5" />
-        <kp value="10000000" />
-        <kd value="10" />
+        <!--mu1 value="2.5" /-->
+        <!--mu2 value="2.5" /-->
+        <!--kp value="1000000" /-->
+        <!--kd value="10" /-->
     </gazebo>
     <!-- Joints -->
@@ -257,8 +253,8 @@
         <parent link="body_link"/>
         <child link="rear_wheel"/>
-        <origin xyz="-0.7 0 -0.3" rpy="0 0 0" />
-        <axis xyz="0 1 0" rpy="0 0 0" />
+        <origin xyz="${-0.5/2+0.05} 0 0" rpy="${-pi/2} 0 0" />
+        <axis xyz="0 0 1" rpy="0 0 0" />
         <!--limit effort="0.4" velocity="12"/-->
-        <dynamics damping="0.1"/>
+        <!--dynamics damping="0.1"/-->
     </joint>
     <!-- Transmissions -->
@@ -277,14 +273,14 @@
         <!-- Collision part -->
         <collision>
-            <origin xyz="0 0 0" rpy="0 ${pi/2} ${pi/2}" />
-            <geometry>
-                <cylinder length="0.1" radius="0.2"/>
+            <origin xyz="0 0 0" rpy="0 0 0" />
+            <geometry>
+                <cylinder length="0.1" radius="0.1"/>
             </geometry>
         </collision>
         <!-- Visual part -->
         <visual>
-            <origin xyz="0 0 0" rpy="0 ${pi/2} ${pi/2}" />
-            <geometry>
-                <cylinder length="0.1" radius="0.2"/>
+            <origin xyz="0 0 0" rpy="0 0 0" />
+            <geometry>
+                <cylinder length="0.1" radius="0.1"/>
             </geometry>
             <material name="black"/>
@@ -292,7 +288,8 @@
         <!-- Inertial part -->
         <inertial>
-            <origin xyz="0 0 0" rpy="0 ${pi/2} ${pi/2}" />
-            <mass value="1"/>
-            <cylinder_inertia mass="1" radius="0.2" height="0.1" />
+            <origin xyz="0 0 0" rpy="0 0 0" />
+            <mass value="1"/>
+            <inertia ixx="0.001" iyy="0.001" izz="0.001" ixy="0" ixz="0" iyz="0" />
+            <!--cylinder_inertia mass="1" radius="0.1" height="0.1" /-->
         </inertial>
     </link>
@@ -302,8 +299,8 @@
             Gazebo/Red
         </material>
-        <mu1 value="200" />
-        <mu2 value="100" />
-        <kp value="10000000" />
-        <kd value="1" />
+        <!--mu1 value="200" /-->
+        <!--mu2 value="100" /-->
+        <!--kp value="1000000" /-->
+        <!--kd value="1" /-->
     </gazebo>
     <!-- Joints -->
@@ -363,8 +360,14 @@
 	<gazebo>
 		<plugin name="gazebo_ros_control" filename="libgazebo_ros_control.so">
-			<robotNamespace>/</robotNamespace>
+			<robotNamespace>/test</robotNamespace>
 			<robotSimType>gazebo_ros_control/DefaultRobotHWSim</robotSimType>
-			<legacyModeNS>true</legacyModeNS>
+			<legacyModeNS>false</legacyModeNS>
 		</plugin>
+        <plugin name="gazebo_ros_joint_state_publisher" filename="libgazebo_ros_joint_state_publisher.so">
+            <robotNamespace>/test</robotNamespace>
+            <jointName>front_wheel_rotate</jointName>
+            <updateRate>50</updateRate>
+            <alwaysOn>true</alwaysOn>
+        </plugin>
 	</gazebo>
 </robot>
