Commit message: Link steer_bot_hardware_gazebo

File: soma_description/urdf/ackermann_macro.xacro (robot description, xacro)
@@ -3,8 +3,9 @@
 https://github.com/benwarrick/simple_ackermann.git -->
 <robot xmlns:xacro="http://www.ros.org/wiki/xacro" name="soma">
-    <!-- Include files -->
-    <include filename="$(find soma_description)/urdf/utils.xacro" />
-    <include filename="$(find soma_description)/urdf/front_wheel_macro.xacro" />
-    <include filename="$(find soma_description)/urdf/rear_wheel_macro.xacro" />
+	<!-- Include files -->
+	<include filename="$(find soma_description)/urdf/utils.xacro" />
+	<include filename="$(find soma_description)/urdf/front_steer_macro.xacro" />
+	<include filename="$(find soma_description)/urdf/front_wheel_macro.xacro" />
+	<include filename="$(find soma_description)/urdf/rear_wheel_macro.xacro" />
 	<!-- Ackermann macro -->
 	<macro name="ackermann_macro" params="parent">
@@ -27,5 +28,5 @@
 				<mass value="${0.8*mass}" />
 				<!-- Inertia matrix of a parallelepiped -->
-                <parallelepiped_inertia mass="${0.8*mass}" width="${width}" height="0.5" depth="${depth}" />
+				<parallelepiped_inertia mass="${0.8*mass}" width="${width}" height="0.5" depth="${depth}" />
 				<!-- Old values: ixx = iyy = izz = 0.001 -->
 			</inertial>
@@ -66,5 +67,5 @@
 				<mass value="${0.19*mass}" />
 				<!-- Inertia matrix of a parallelepiped -->
-                <parallelepiped_inertia mass="${0.19*mass}" width="0.85" height="0.9" depth="${depth}" />
+				<parallelepiped_inertia mass="${0.19*mass}" width="0.85" height="0.9" depth="${depth}" />
 				<!-- Old values: ixx = iyy = izz = 0.001 -->
 			</inertial>
@@ -105,5 +106,5 @@
 				<mass value="${0.01*mass}" />
 				<!-- Inertia matrix of a parallelepiped -->
-                <parallelepiped_inertia mass="${0.01*mass}" width="0.05" height="0.3" depth="0.05" />
+				<parallelepiped_inertia mass="${0.01*mass}" width="0.05" height="0.3" depth="0.05" />
 				<!-- Old values: ixx = iyy = izz = 0.001 -->
 			</inertial>
@@ -132,11 +133,11 @@
 		</gazebo>
 		<!-- Build links and joints for ackermann_steering_controller -->
-		<!--front_wheel_macro parent="body_bottom_link" prefix="ackermann" xyz="${width/2 + 0.5} 0 ${-0.5/2}" /-->
-		<!--rear_wheel_macro parent="body_bottom_link" prefix="ackermann" xyz="${-width/2 - 0.5} 0 ${-0.5/2}" /-->
-        <!-- Build wheels -->
-        <front_wheel_macro parent="body_bottom_link" prefix="left" xyz="${width/2} ${depth/2 + 0.0889} -0.2" />
-        <front_wheel_macro parent="body_bottom_link" prefix="right" xyz="${width/2} ${-depth/2 - 0.0889} -0.2" />
-        <rear_wheel_macro parent="body_bottom_link" prefix="left" xyz="${-width/2} ${depth/2 + 0.0889} -0.2" />
-        <rear_wheel_macro parent="body_bottom_link" prefix="right" xyz="${-width/2} ${-depth/2 - 0.0889} -0.2" />
-    </macro>
+		<front_steer_macro parent="body_bottom_link" prefix="ackermann" xyz="${width/2} 0 ${-0.5/2}" />
+		<rear_wheel_macro parent="body_bottom_link" prefix="ackermann" xyz="${-width/2} 0 ${-0.5/2}" />
+		<!-- Build wheels -->
+		<front_wheel_macro parent="body_bottom_link" prefix="left" xyz="${width/2} ${depth/2 + 0.0889} ${-0.5/2}" />
+		<front_wheel_macro parent="body_bottom_link" prefix="right" xyz="${width/2} ${-depth/2 - 0.0889} ${-0.5/2}" />
+		<rear_wheel_macro parent="body_bottom_link" prefix="left" xyz="${-width/2} ${depth/2 + 0.0889} ${-0.5/2}" />
+		<rear_wheel_macro parent="body_bottom_link" prefix="right" xyz="${-width/2} ${-depth/2 - 0.0889} ${-0.5/2}" />
+	</macro>
 </robot>

File: soma_description/urdf/front_wheel_macro.xacro (robot description, xacro)
@@ -2,10 +2,10 @@
 <robot xmlns:xacro="http://www.ros.org/wiki/xacro" name="soma">
     <!-- Front wheel macro -->
-	<macro name="front_wheel_macro" params="parent prefix xyz">
-		<!-- General properties used for inertia computation -->
-		<property name="mass" value="12" />
-		<property name="radius" value="0.2286" />
-		<property name="length" value="0.0889" />
-		<!-- Joints -->
+    <macro name="front_wheel_macro" params="parent prefix xyz">
+        <!-- General properties used for inertia computation -->
+        <property name="mass" value="12" />
+        <property name="radius" value="0.2286" />
+        <property name="length" value="0.0889" />
+        <!-- Joints -->
         <joint name="${prefix}_front_wheel_hinge" type="revolute">
             <parent link="${parent}"/>
@@ -20,9 +20,9 @@
             <parent link="${prefix}_front_wheel_assembly"/>
             <child link="${prefix}_front_wheel"/>
-            <origin xyz="0.0 0.0 0.0" rpy="0 0 0" />
-            <axis xyz="0 1 0" rpy="0 0 0" />
+            <origin xyz="0.0 0.0 0.0" rpy="${-pi/2} 0 0" />
+            <axis xyz="0 0 1" rpy="0 0 0" />
             <dynamics damping="0.1"/>
         </joint>
-		<!-- Transmissions -->
+        <!-- Transmissions -->
         <transmission name="${prefix}_front_wheel_hinge_trans">
             <type>transmission_interface/SimpleTransmission</type>
@@ -45,9 +45,9 @@
             </actuator>
         </transmission>
-		<!-- Links -->
+        <!-- Links -->
         <link name="${prefix}_front_wheel">
             <!-- Collision part -->
             <collision>
-                <origin xyz="0 0 0" rpy="0 ${pi/2} ${pi/2}" />
+                <origin xyz="0 0 0" rpy="0 0 0" />
                 <geometry>
                     <cylinder length="${length}" radius="${radius}"/>
@@ -56,5 +56,5 @@
             <!-- Visual part -->
             <visual>
-                <origin xyz="0 0 0" rpy="0 ${pi/2} ${pi/2}" />
+                <origin xyz="0 0 0" rpy="0 0 0" />
                 <geometry>
                     <cylinder length="${length}" radius="${radius}"/>
@@ -64,5 +64,5 @@
             <!-- Inertial part -->
             <inertial>
-                <origin xyz="0 0 0" rpy="0 ${pi/2} ${pi/2}" />
+                <origin xyz="0 0 0" rpy="0 0 0" />
                 <mass value="${mass}"/>
                 <cylinder_inertia mass="${mass}" radius="${radius}" height="${length}" />
@@ -72,14 +72,14 @@
             <!-- Collision part -->
             <collision>
-                <origin xyz="0 0 0" rpy="0 ${pi/2} ${pi/2}" />
+                <origin xyz="0 0 0.3" rpy="0 0 0" />
                 <geometry>
-                    <cylinder length="0.001" radius="0.04"/>
+                    <cylinder length="0.05" radius="0.1"/>
                 </geometry>
             </collision>
             <!-- Visual part -->
             <visual>
-                <origin xyz="0 0 0" rpy="0 ${pi/2} ${pi/2}" />
+                <origin xyz="0 0 0.3" rpy="0 0 0" />
                 <geometry>
-                    <cylinder length="0.001" radius="0.04"/>
+                    <cylinder length="0.05" radius="0.1"/>
                 </geometry>
                 <material name="white"/>
@@ -87,29 +87,29 @@
             <!-- Inertial part -->
             <inertial>
-                <origin xyz="0 0 0" rpy="0 ${pi/2} ${pi/2}" />
+                <origin xyz="0 0 0.3" rpy="0 0 0" />
                 <mass value="0.2"/>
-                <cylinder_inertia mass="0.2" radius="0.3" height="0.1"/>
+                <cylinder_inertia mass="0.2" radius="0.1" height="0.05"/>
             </inertial>
         </link>
-		<!-- Gazebo additional parameters -->
-		<gazebo reference="${prefix}_front_wheel">
-			<material>
+        <!-- Gazebo additional parameters -->
+        <gazebo reference="${prefix}_front_wheel">
+            <material>
 				Gazebo/Red
-			</material>
-			<mu1 value="200" />
-			<mu2 value="200" />
-			<kp value="1000000" />
-			<kd value="10" />
-		</gazebo>
+            </material>
+            <mu1 value="200" />
+            <mu2 value="200" />
+            <kp value="1000000" />
+            <kd value="10" />
+        </gazebo>
         <gazebo reference="${prefix}_front_wheel_assembly">
-			<material>
+            <material>
 				Gazebo/Red
-			</material>
-			<mu1 value="200" />
-			<mu2 value="200" />
-			<kp value="1000000" />
-			<kd value="10" />
-		</gazebo>
-	</macro>
-	<!-- END front wheel macro -->
+            </material>
+            <mu1 value="200" />
+            <mu2 value="200" />
+            <kp value="1000000" />
+            <kd value="10" />
+        </gazebo>
+    </macro>
+    <!-- END front wheel macro -->
 </robot>

File: soma_description/urdf/rear_wheel_macro.xacro (robot description, xacro)
@@ -2,15 +2,15 @@
 <robot xmlns:xacro="http://www.ros.org/wiki/xacro" name="soma">
     <!-- Rear wheel macro -->
-	<macro name="rear_wheel_macro" params="parent prefix xyz">
-		<!-- General properties used for inertia computation -->
-		<property name="mass" value="12" />
-		<property name="radius" value="0.2286" />
-		<property name="length" value="0.0889" />
-		<!-- Joint -->
+    <macro name="rear_wheel_macro" params="parent prefix xyz">
+        <!-- General properties used for inertia computation -->
+        <property name="mass" value="12" />
+        <property name="radius" value="0.2286" />
+        <property name="length" value="0.0889" />
+        <!-- Joint -->
         <joint name="${prefix}_rear_wheel_rotate" type="continuous">
             <parent link="${parent}"/>
             <child link="${prefix}_rear_wheel"/>
-            <origin xyz="${xyz}" rpy="0 0 0" />
-            <axis xyz="0 1 0" rpy="0 0 0" />
+            <origin xyz="${xyz}" rpy="${-pi/2} 0 0" />
+            <axis xyz="0 0 1" rpy="0 0 0" />
             <!--limit effort="0.4" velocity="12"/-->
             <dynamics damping="0.1"/>
@@ -27,9 +27,9 @@
             </actuator>
         </transmission>
-		<!-- Link -->
+        <!-- Link -->
         <link name="${prefix}_rear_wheel">
             <!-- Collision part -->
             <collision>
-                <origin xyz="0 0 0" rpy="0 ${pi/2} ${pi/2}" />
+                <origin xyz="0 0 0" rpy="0 0 0" />
                 <geometry>
                     <cylinder length="${length}" radius="${radius}"/>
@@ -38,5 +38,5 @@
             <!-- Visual part -->
             <visual>
-                <origin xyz="0 0 0" rpy="0 ${pi/2} ${pi/2}" />
+                <origin xyz="0 0 0" rpy="0 0 0" />
                 <geometry>
                     <cylinder length="${length}" radius="${radius}"/>
@@ -46,20 +46,20 @@
             <!-- Inertial part -->
             <inertial>
-                <origin xyz="0 0 0" rpy="0 ${pi/2} ${pi/2}" />
+                <origin xyz="0 0 0" rpy="0 0 0" />
                 <mass value="${mass}"/>
                 <cylinder_inertia mass="${mass}" radius="${radius}" height="${length}" />
             </inertial>
         </link>
-		<!-- Gazebo additional parameters -->
-		<gazebo reference="${prefix}_rear_wheel">
-			<material>
+        <!-- Gazebo additional parameters -->
+        <gazebo reference="${prefix}_rear_wheel">
+            <material>
 				Gazebo/Red
-			</material>
-			<mu1 value="2.5" />
-			<mu2 value="2.5" />
-			<kp value="1000000" />
-			<kd value="10" />
-		</gazebo>
-	</macro>
-	<!-- END rear wheel macro -->
+            </material>
+            <mu1 value="2.5" />
+            <mu2 value="2.5" />
+            <kp value="1000000" />
+            <kd value="10" />
+        </gazebo>
+    </macro>
+    <!-- END rear wheel macro -->
 </robot>

File: soma_description/urdf/soma.urdf.xacro (robot description, xacro)
@@ -10,26 +10,28 @@
 	<ackermann_macro parent="base_link" />
 	<!-- Build Velodyne -->
-	<!--VLP-16 parent="body_bottom_link" name="velodyne" topic="/velodyne_points">
+	<!-- <VLP-16 parent="body_bottom_link" name="velodyne" topic="/velodyne_points">
 		<origin xyz="0.075 0.0 ${1.70 - 0.25}" rpy="0.0 0.0 0.0" />
-	</VLP-16-->
+	</VLP-16> -->
 	<!-- Build IMU -->
-	<!--imu_macro parent="body_bottom_link">
+	<!-- <imu_macro parent="body_bottom_link">
 		<origin xyz="${-0.525 + 0.05/2} 0.0 ${1.40 - 0.25 + 0.025/2}" rpy="0.0 0.0 0.0" />
-	</imu_macro-->
+	</imu_macro> -->
 	<!-- Build Realsense -->
 	<!-- Front -->
-	<!--realsense_macro parent="body_bottom_link" prefix="f">
+	<!-- <realsense_macro parent="body_bottom_link" prefix="f">
 		<origin xyz="0.325 0.0 ${1.10 - 0.25}" rpy="0.0 0.0 0.0" />
-	</realsense_macro-->
+	</realsense_macro> -->
 	<!-- Rear -->
-	<!--realsense_macro parent="body_bottom_link" prefix="r">
+	<!-- <realsense_macro parent="body_bottom_link" prefix="r">
 		<origin xyz="-0.525 0.0 ${1.10 - 0.25}" rpy="0.0 0.0 ${-pi}" />
-	</realsense_macro-->
+	</realsense_macro> -->
 	<!-- Gazebo plugins -->
 	<gazebo>
+		<!-- Load ros_control plugin using the steer_bot_hardware_gazebo
+   		implementation of the hardware_interface::RobotHW -->
 		<plugin name="gazebo_ros_control" filename="libgazebo_ros_control.so">
-			<robotNamespace>/</robotNamespace>
-			<robotSimType>gazebo_ros_control/DefaultRobotHWSim</robotSimType>
-			<legacyModeNS>true</legacyModeNS>
+			<robotNamespace>/soma</robotNamespace>
+			<robotSimType>steer_bot_hardware_gazebo/SteerBotHardwareGazebo</robotSimType>
+			<legacyModeNS>false</legacyModeNS>
 		</plugin>
 	</gazebo>

Commit message: Add virtual_rear_wheel macro

File: soma_description/urdf/ackermann_macro.xacro (robot description, xacro)
@@ -8,4 +8,5 @@
 	<include filename="$(find soma_description)/urdf/front_wheel_macro.xacro" />
 	<include filename="$(find soma_description)/urdf/rear_wheel_macro.xacro" />
+	<include filename="$(find soma_description)/urdf/virtual_rear_wheel_macro.xacro" />
 	<!-- Ackermann macro -->
 	<macro name="ackermann_macro" params="parent">
@@ -134,5 +135,5 @@
 		<!-- Build links and joints for ackermann_steering_controller -->
 		<front_steer_macro parent="body_bottom_link" prefix="ackermann" xyz="${width/2} 0 ${-0.5/2}" />
-		<rear_wheel_macro parent="body_bottom_link" prefix="ackermann" xyz="${-width/2} 0 ${-0.5/2}" />
+		<virtual_rear_wheel_macro parent="body_bottom_link" prefix="ackermann" xyz="${-width/2} 0 ${-0.5/2}" />
 		<!-- Build wheels -->
 		<front_wheel_macro parent="body_bottom_link" prefix="left" xyz="${width/2} ${depth/2 + 0.0889} ${-0.5/2}" />

File: soma_description/urdf/front_steer_macro.xacro (robot description, xacro)
@@ -54,17 +54,8 @@
 				Gazebo/Red
             </material>
-            <mu1 value="200" />
-            <mu2 value="200" />
-            <kp value="1000000" />
-            <kd value="10" />
-        </gazebo>
-        <gazebo reference="${prefix}_front_steer">
-            <material>
-				Gazebo/Red
-            </material>
-            <mu1 value="200" />
-            <mu2 value="200" />
-            <kp value="1000000" />
-            <kd value="10" />
+            <!-- <mu1 value="200" /> -->
+            <!-- <mu2 value="200" /> -->
+            <!-- <kp value="1000000" /> -->
+            <!-- <kd value="10" /> -->
         </gazebo>
     </macro>

File: soma_description/urdf/front_wheel_macro.xacro (robot description, xacro)
@@ -97,8 +97,8 @@
 				Gazebo/Red
             </material>
-            <mu1 value="200" />
-            <mu2 value="200" />
-            <kp value="1000000" />
-            <kd value="10" />
+            <!-- <mu1 value="200" /> -->
+            <!-- <mu2 value="200" /> -->
+            <!-- <kp value="1000000" /> -->
+            <!-- <kd value="10" /> -->
         </gazebo>
         <gazebo reference="${prefix}_front_wheel_assembly">
@@ -106,8 +106,8 @@
 				Gazebo/Red
             </material>
-            <mu1 value="200" />
-            <mu2 value="200" />
-            <kp value="1000000" />
-            <kd value="10" />
+            <!-- <mu1 value="200" /> -->
+            <!-- <mu2 value="200" /> -->
+            <!-- <kp value="1000000" /> -->
+            <!-- <kd value="10" /> -->
         </gazebo>
     </macro>

File: soma_description/urdf/virtual_rear_wheel_macro.xacro (robot description, xacro)
@@ -2,5 +2,5 @@
 <robot xmlns:xacro="http://www.ros.org/wiki/xacro" name="soma">
     <!-- Rear wheel macro -->
-    <macro name="rear_wheel_macro" params="parent prefix xyz">
+    <macro name="virtual_rear_wheel_macro" params="parent prefix xyz">
         <!-- General properties used for inertia computation -->
         <property name="mass" value="12" />
@@ -8,7 +8,7 @@
         <property name="length" value="0.0889" />
         <!-- Joint -->
-        <joint name="${prefix}_rear_wheel_rotate" type="continuous">
+        <joint name="${prefix}_virtual_rear_wheel_rotate" type="continuous">
             <parent link="${parent}"/>
-            <child link="${prefix}_rear_wheel"/>
+            <child link="${prefix}_virtual_rear_wheel"/>
             <origin xyz="${xyz}" rpy="${-pi/2} 0 0" />
             <axis xyz="0 0 1" rpy="0 0 0" />
@@ -17,10 +17,10 @@
         </joint>
         <!-- Transmission -->
-        <transmission name="${prefix}_rear_wheel_rotate_trans">
+        <transmission name="${prefix}_virtual_rear_wheel_rotate_trans">
             <type>transmission_interface/SimpleTransmission</type>
-            <joint name="${prefix}_rear_wheel_rotate">
+            <joint name="${prefix}_virtual_rear_wheel_rotate">
                 <hardwareInterface>hardware_interface/VelocityJointInterface</hardwareInterface>
             </joint>
-            <actuator name="${prefix}_rear_wheel_rotate_motor">
+            <actuator name="${prefix}_virtual_rear_wheel_rotate_motor">
                 <hardwareInterface>hardware_interface/VelocityJointInterface</hardwareInterface>
                 <mechanicalReduction>1</mechanicalReduction>
@@ -28,14 +28,14 @@
         </transmission>
         <!-- Link -->
-        <link name="${prefix}_rear_wheel">
+        <link name="${prefix}_virtual_rear_wheel">
             <!-- Collision part -->
-            <collision>
+            <!-- <collision>
                 <origin xyz="0 0 0" rpy="0 0 0" />
                 <geometry>
                     <cylinder length="${length}" radius="${radius}"/>
                 </geometry>
-            </collision>
+            </collision> -->
             <!-- Visual part -->
-            <visual>
+            <!-- <visual>
                 <origin xyz="0 0 0" rpy="0 0 0" />
                 <geometry>
@@ -43,14 +43,14 @@
                 </geometry>
                 <material name="black"/>
-            </visual>
+            </visual> -->
             <!-- Inertial part -->
-            <inertial>
+            <!-- <inertial>
                 <origin xyz="0 0 0" rpy="0 0 0" />
                 <mass value="${mass}"/>
                 <cylinder_inertia mass="${mass}" radius="${radius}" height="${length}" />
-            </inertial>
+            </inertial> -->
         </link>
         <!-- Gazebo additional parameters -->
-        <gazebo reference="${prefix}_rear_wheel">
+        <gazebo reference="${prefix}_virtual_rear_wheel">
             <material>
 				Gazebo/Red
