Commit message: Introduce notations

File: soma_description/urdf/ackermann_macro.xacro (robot description, xacro)
@@ -20,5 +20,5 @@
 			<parent link="${parent}" />
 			<child link="body_bottom_link" />
-			<origin xyz="0 0 ${0.2286 + 0.5/2}" rpy="0.0 0.0 0.0" />
+			<origin xyz="0 0 ${0.2286 + 0.5/4}" rpy="0.0 0.0 0.0" />
 		</joint>
 		<!-- Bottom body link -->
@@ -55,90 +55,12 @@
 			</material>
 		</gazebo>
-		<!-- Middle body joint -->
-		<joint name="body_middle_joint" type="fixed">
-			<parent link="${parent}" />
-			<child link="body_middle_link" />
-			<origin xyz="-0.1 0 ${0.2286 + 0.5 + 0.9/2}" rpy="0.0 0.0 0.0" />
-		</joint>
-		<!-- Middle body link -->
-		<link name="body_middle_link">
-			<!-- Inertial part -->
-			<inertial>
-				<origin xyz="0.0 0.0 0.0" rpy="0.0 0.0 0.0" />
-				<mass value="${0.19*mass}" />
-				<!-- Inertia matrix of a parallelepiped -->
-				<parallelepiped_inertia mass="${0.19*mass}" width="0.85" height="0.9" depth="${depth}" />
-				<!-- Old values: ixx = iyy = izz = 0.001 -->
-			</inertial>
-			<!-- Visual part -->
-			<visual>
-				<origin xyz="0.0 0.0 0.0" rpy="0.0 0.0 0.0" />
-				<geometry>
-					<box size="0.85 ${depth} 0.9" />
-				</geometry>
-				<material name="gray" />
-			</visual>
-			<!-- Collision part -->
-			<collision>
-				<origin xyz="0.0 0.0 0.0" rpy="0.0 0.0 0.0" />
-				<geometry>
-					<box size="0.85 ${depth} 0.9" />
-				</geometry>
-			</collision>
-		</link>
-		<!-- END middle body link -->
-		<!-- Gazebo additional parameters -->
-		<gazebo reference="body_middle_link">
-			<material>
-				Gazebo/Gray
-			</material>
-		</gazebo>
-		<!-- Top body joint -->
-		<joint name="body_top_joint" type="fixed">
-			<parent link="${parent}" />
-			<child link="body_top_link" />
-			<origin xyz="0.075 0 ${0.2286 + 0.5 + 0.9 + 0.3/2}" rpy="0.0 0.0 0.0" />
-		</joint>
-		<!-- Top body link -->
-		<link name="body_top_link">
-			<!-- Inertial part -->
-			<inertial>
-				<origin xyz="0.0 0.0 0.0" rpy="0.0 0.0 0.0" />
-				<mass value="${0.01*mass}" />
-				<!-- Inertia matrix of a parallelepiped -->
-				<parallelepiped_inertia mass="${0.01*mass}" width="0.05" height="0.3" depth="0.05" />
-				<!-- Old values: ixx = iyy = izz = 0.001 -->
-			</inertial>
-			<!-- Visual part -->
-			<visual>
-				<origin xyz="0.0 0.0 0.0" rpy="0.0 0.0 0.0" />
-				<geometry>
-					<box size="0.05 0.05 0.3" />
-				</geometry>
-				<material name="gray" />
-			</visual>
-			<!-- Collision part -->
-			<collision>
-				<origin xyz="0.0 0.0 0.0" rpy="0.0 0.0 0.0" />
-				<geometry>
-					<box size="0.05 0.05 0.3" />
-				</geometry>
-			</collision>
-		</link>
-		<!-- END top body link -->
-		<!-- Gazebo additional parameters -->
-		<gazebo reference="body_top_link">
-			<material>
-				Gazebo/Gray
-			</material>
-		</gazebo>
 		<!-- Build links and joints for ackermann_steering_controller -->
-		<front_steer_macro parent="body_bottom_link" prefix="ackermann" xyz="${width/2} 0 ${-0.5/2}" />
-		<virtual_rear_wheel_macro parent="body_bottom_link" prefix="ackermann" xyz="${-width/2} 0 ${-0.5/2}" />
+		<front_steer_macro parent="body_bottom_link" prefix="ackermann" xyz="${width/2 - 0.1} 0 ${-0.5/4}" />
+		<virtual_rear_wheel_macro parent="body_bottom_link" prefix="ackermann" xyz="${-width/2 + 0.1} 0 ${-0.5/4}" />
 		<!-- Build wheels -->
-		<front_wheel_macro parent="body_bottom_link" prefix="left" xyz="${width/2} ${depth/2 + 0.0889} ${-0.5/2}" />
-		<front_wheel_macro parent="body_bottom_link" prefix="right" xyz="${width/2} ${-depth/2 - 0.0889} ${-0.5/2}" />
-		<rear_wheel_macro parent="body_bottom_link" prefix="left" xyz="${-width/2} ${depth/2 + 0.0889} ${-0.5/2}" />
-		<rear_wheel_macro parent="body_bottom_link" prefix="right" xyz="${-width/2} ${-depth/2 - 0.0889} ${-0.5/2}" />
+		<front_wheel_macro parent="body_bottom_link" prefix="left" xyz="${width/2 - 0.1} ${depth/2 + 0.0889} ${-0.5/4}" />
+		<front_wheel_macro parent="body_bottom_link" prefix="right" xyz="${width/2 - 0.1} ${-depth/2 - 0.0889} ${-0.5/4}" />
+		<rear_wheel_macro parent="body_bottom_link" prefix="left" xyz="${-width/2 + 0.1} ${depth/2 + 0.0889} ${-0.5/4}" />
+		<rear_wheel_macro parent="body_bottom_link" prefix="right" xyz="${-width/2 + 0.1} ${-depth/2 - 0.0889} ${-0.5/4}" />
 	</macro>
 </robot>

File: soma_description/urdf/front_steer_macro.xacro (robot description, xacro)
@@ -12,5 +12,5 @@
             <!-- <limit effort="0.4" velocity="1" lower="-1" upper="1"/> -->
             <limit effort="10" velocity="5" lower="-0.2" upper="0.2"/>
-            <dynamics damping="0.1"/>
+            <!-- <dynamics damping="0.1"/> -->
         </joint>
         <!-- Initial values: effort=0.4 velocity=12 -->

File: soma_description/urdf/front_wheel_macro.xacro (robot description, xacro)
@@ -15,5 +15,5 @@
             <!-- <limit effort="0.4" velocity="1" lower="-1" upper="1"/> -->
             <limit effort="10" velocity="5" lower="-0.2" upper="0.2"/>
-            <dynamics damping="0.1"/>
+            <!-- <dynamics damping="0.1"/> -->
         </joint>
         <!-- Initial values: effort=0.4 velocity=12 -->

File: soma_description/urdf/virtual_rear_wheel_macro.xacro (robot description, xacro)
@@ -14,5 +14,5 @@
             <axis xyz="0 0 1" rpy="0 0 0" />
             <!--limit effort="0.4" velocity="12"/-->
-            <dynamics damping="0.1"/>
+            <!-- <dynamics damping="0.1"/> -->
         </joint>
         <!-- Transmission -->

Commit message: Ackermann steering working

File: soma_description/urdf/ackermann_macro.xacro (robot description, xacro)
@@ -20,5 +20,5 @@
 			<parent link="${parent}" />
 			<child link="body_bottom_link" />
-			<origin xyz="0 0 ${0.2286 + 0.5/4}" rpy="0.0 0.0 0.0" />
+			<origin xyz="0 0 ${0.2286 + 0.5/2}" rpy="0.0 0.0 0.0" />
 		</joint>
 		<!-- Bottom body link -->
@@ -55,12 +55,90 @@
 			</material>
 		</gazebo>
+		<!-- Middle body joint -->
+		<joint name="body_middle_joint" type="fixed">
+			<parent link="${parent}" />
+			<child link="body_middle_link" />
+			<origin xyz="-0.1 0 ${0.2286 + 0.5 + 0.9/2}" rpy="0.0 0.0 0.0" />
+		</joint>
+		<!-- Middle body link -->
+		<link name="body_middle_link">
+			<!-- Inertial part -->
+			<inertial>
+				<origin xyz="0.0 0.0 0.0" rpy="0.0 0.0 0.0" />
+				<mass value="${0.19*mass}" />
+				<!-- Inertia matrix of a parallelepiped -->
+				<parallelepiped_inertia mass="${0.19*mass}" width="0.85" height="0.9" depth="${depth}" />
+				<!-- Old values: ixx = iyy = izz = 0.001 -->
+			</inertial>
+			<!-- Visual part -->
+			<visual>
+				<origin xyz="0.0 0.0 0.0" rpy="0.0 0.0 0.0" />
+				<geometry>
+					<box size="0.85 ${depth} 0.9" />
+				</geometry>
+				<material name="gray" />
+			</visual>
+			<!-- Collision part -->
+			<collision>
+				<origin xyz="0.0 0.0 0.0" rpy="0.0 0.0 0.0" />
+				<geometry>
+					<box size="0.85 ${depth} 0.9" />
+				</geometry>
+			</collision>
+		</link>
+		<!-- END middle body link -->
+		<!-- Gazebo additional parameters -->
+		<gazebo reference="body_middle_link">
+			<material>
+						Gazebo/Gray
+			</material>
+		</gazebo>
+		<!-- Top body joint -->
+		<joint name="body_top_joint" type="fixed">
+			<parent link="${parent}" />
+			<child link="body_top_link" />
+			<origin xyz="0.075 0 ${0.2286 + 0.5 + 0.9 + 0.3/2}" rpy="0.0 0.0 0.0" />
+		</joint>
+		<!-- Top body link -->
+		<link name="body_top_link">
+			<!-- Inertial part -->
+			<inertial>
+				<origin xyz="0.0 0.0 0.0" rpy="0.0 0.0 0.0" />
+				<mass value="${0.01*mass}" />
+				<!-- Inertia matrix of a parallelepiped -->
+				<parallelepiped_inertia mass="${0.01*mass}" width="0.05" height="0.3" depth="0.05" />
+				<!-- Old values: ixx = iyy = izz = 0.001 -->
+			</inertial>
+			<!-- Visual part -->
+			<visual>
+				<origin xyz="0.0 0.0 0.0" rpy="0.0 0.0 0.0" />
+				<geometry>
+					<box size="0.05 0.05 0.3" />
+				</geometry>
+				<material name="gray" />
+			</visual>
+			<!-- Collision part -->
+			<collision>
+				<origin xyz="0.0 0.0 0.0" rpy="0.0 0.0 0.0" />
+				<geometry>
+					<box size="0.05 0.05 0.3" />
+				</geometry>
+			</collision>
+		</link>
+		<!-- END top body link -->
+		<!-- Gazebo additional parameters -->
+		<gazebo reference="body_top_link">
+			<material>
+						Gazebo/Gray
+			</material>
+		</gazebo>
 		<!-- Build links and joints for ackermann_steering_controller -->
-		<front_steer_macro parent="body_bottom_link" prefix="ackermann" xyz="${width/2 - 0.1} 0 ${-0.5/4}" />
-		<virtual_rear_wheel_macro parent="body_bottom_link" prefix="ackermann" xyz="${-width/2 + 0.1} 0 ${-0.5/4}" />
+		<front_steer_macro parent="body_bottom_link" prefix="ackermann" xyz="${width/2} 0 ${-0.5/2}" />
+		<virtual_rear_wheel_macro parent="body_bottom_link" prefix="ackermann" xyz="${-width/2} 0 ${-0.5/2}" />
 		<!-- Build wheels -->
-		<front_wheel_macro parent="body_bottom_link" prefix="left" xyz="${width/2 - 0.1} ${depth/2 + 0.0889} ${-0.5/4}" />
-		<front_wheel_macro parent="body_bottom_link" prefix="right" xyz="${width/2 - 0.1} ${-depth/2 - 0.0889} ${-0.5/4}" />
-		<rear_wheel_macro parent="body_bottom_link" prefix="left" xyz="${-width/2 + 0.1} ${depth/2 + 0.0889} ${-0.5/4}" />
-		<rear_wheel_macro parent="body_bottom_link" prefix="right" xyz="${-width/2 + 0.1} ${-depth/2 - 0.0889} ${-0.5/4}" />
+		<front_wheel_macro parent="body_bottom_link" prefix="left" xyz="${width/2} ${depth/2 + 0.0889} ${-0.5/2}" />
+		<front_wheel_macro parent="body_bottom_link" prefix="right" xyz="${width/2} ${-depth/2 - 0.0889} ${-0.5/2}" />
+		<rear_wheel_macro parent="body_bottom_link" prefix="left" xyz="${-width/2} ${depth/2 + 0.0889} ${-0.5/2}" />
+		<rear_wheel_macro parent="body_bottom_link" prefix="right" xyz="${-width/2} ${-depth/2 - 0.0889} ${-0.5/2}" />
 	</macro>
 </robot>

File: soma_description/urdf/front_steer_macro.xacro (robot description, xacro)
@@ -12,5 +12,5 @@
             <!-- <limit effort="0.4" velocity="1" lower="-1" upper="1"/> -->
             <limit effort="10" velocity="5" lower="-0.2" upper="0.2"/>
-            <!-- <dynamics damping="0.1"/> -->
+            <dynamics damping="0.1"/>
         </joint>
         <!-- Initial values: effort=0.4 velocity=12 -->
@@ -55,12 +55,8 @@
 				Gazebo/Red
             </material>
-            <!-- <mu1 value="200" /> -->
-            <!-- <mu2 value="200" /> -->
-            <!-- <kp value="1000000" /> -->
-            <!-- <kd value="10" /> -->
         </gazebo>
-        <gazebo reference="${prefix}_front_steer_hinge">
+        <!-- <gazebo reference="${prefix}_front_steer_hinge">
             <provideFeedback>true</provideFeedback>
-        </gazebo>
+        </gazebo> -->
     </macro>
     <!-- END front wheel macro -->

File: soma_description/urdf/front_wheel_macro.xacro (robot description, xacro)
@@ -4,5 +4,5 @@
     <macro name="front_wheel_macro" params="parent prefix xyz">
         <!-- General properties used for inertia computation -->
-        <property name="mass" value="12" />
+        <property name="mass" value="1" />
         <property name="radius" value="0.2286" />
         <property name="length" value="0.0889" />
@@ -15,5 +15,5 @@
             <!-- <limit effort="0.4" velocity="1" lower="-1" upper="1"/> -->
             <limit effort="10" velocity="5" lower="-0.2" upper="0.2"/>
-            <!-- <dynamics damping="0.1"/> -->
+            <dynamics damping="0.1"/>
         </joint>
         <!-- Initial values: effort=0.4 velocity=12 -->
@@ -23,5 +23,6 @@
             <origin xyz="0.0 0.0 0.0" rpy="${-pi/2} 0 0" />
             <axis xyz="0 0 1" rpy="0 0 0" />
-            <!-- <dynamics damping="0.1"/> -->
+            <limit effort="10" velocity="5"/>
+            <dynamics damping="0.1"/>
         </joint>
         <!-- Transmissions -->
@@ -100,6 +101,6 @@
             <!-- <mu1 value="200" /> -->
             <!-- <mu2 value="200" /> -->
-            <!-- <kp value="1000000" /> -->
-            <!-- <kd value="10" /> -->
+            <kp value="1000000000" />
+            <kd value="1" />
         </gazebo>
         <gazebo reference="${prefix}_front_wheel_assembly">
@@ -107,8 +108,8 @@
 				Gazebo/Red
             </material>
-            <!-- <mu1 value="200" /> -->
-            <!-- <mu2 value="200" /> -->
-            <!-- <kp value="1000000" /> -->
-            <!-- <kd value="10" /> -->
+            <mu1 value="0.5" />
+            <mu2 value="0.5" />
+            <kp value="1000000000" />
+            <kd value="10" />
         </gazebo>
     </macro>

File: soma_description/urdf/rear_wheel_macro.xacro (robot description, xacro)
@@ -4,5 +4,5 @@
     <macro name="rear_wheel_macro" params="parent prefix xyz">
         <!-- General properties used for inertia computation -->
-        <property name="mass" value="12" />
+        <property name="mass" value="1" />
         <property name="radius" value="0.2286" />
         <property name="length" value="0.0889" />
@@ -13,6 +13,6 @@
             <origin xyz="${xyz}" rpy="${-pi/2} 0 0" />
             <axis xyz="0 0 1" rpy="0 0 0" />
-            <!--limit effort="0.4" velocity="12"/-->
-            <!-- <dynamics damping="0.1"/> -->
+            <limit effort="10" velocity="5"/>
+            <dynamics damping="0.1"/>
         </joint>
         <!-- Transmission -->
@@ -56,8 +56,8 @@
 				Gazebo/Red
             </material>
-            <!-- <mu1 value="200" /> -->
-            <!-- <mu2 value="200" /> -->
-            <!-- <kp value="1000000" /> -->
-            <!-- <kd value="10" /> -->
+            <mu1 value="0.5" />
+            <mu2 value="0.5" />
+            <kp value="1000000000" />
+            <kd value="10" />
         </gazebo>
     </macro>

File: soma_description/urdf/sensors_macro.xacro (robot description, xacro)
@@ -23,7 +23,5 @@
 				<mass value="${mass}" />
 				<!-- Inertia matrix of a parallelepiped -->
-				<inertia ixx="${mass / 12 * (depth ** 2 + height ** 2)}" ixy="0.0"
-						 ixz="0.0" iyy="${mass / 12 * (width ** 2 + height ** 2)}"
-						 iyz="0.0" izz="${mass / 12 * (width ** 2 + depth ** 2)}" />
+				<inertia ixx="${mass / 12 * (depth ** 2 + height ** 2)}" ixy="0.0" ixz="0.0" iyy="${mass / 12 * (width ** 2 + height ** 2)}" iyz="0.0" izz="${mass / 12 * (width ** 2 + depth ** 2)}" />
 			</inertial>
 			<!-- Visual part -->
@@ -49,23 +47,23 @@
 				Gazebo/Red
 			</material>
-    		<gravity>true</gravity>
-    		<sensor name="imu_sensor" type="imu">
-      			<always_on>true</always_on>
-      			<update_rate>100</update_rate>
-      			<visualize>true</visualize>
-      			<topic>__default_topic__</topic>
-      			<plugin filename="libgazebo_ros_imu_sensor.so" name="imu_plugin">
-        			<topicName>imu</topicName>
-        			<bodyName>imu_link</bodyName>
-        			<updateRateHZ>10.0</updateRateHZ>
-        			<gaussianNoise>0.0</gaussianNoise>
-        			<xyzOffset>0 0 0</xyzOffset>
-        			<rpyOffset>0 0 0</rpyOffset>
-        			<frameName>imu_link</frameName>
-        			<initialOrientationAsReference>false</initialOrientationAsReference>
-      			</plugin>
-      			<pose>0 0 0 0 0 0</pose>
-    		</sensor>
-  		</gazebo>
+			<gravity>true</gravity>
+			<sensor name="imu_sensor" type="imu">
+				<always_on>true</always_on>
+				<update_rate>100</update_rate>
+				<visualize>true</visualize>
+				<topic>__default_topic__</topic>
+				<plugin filename="libgazebo_ros_imu_sensor.so" name="imu_plugin">
+					<topicName>imu</topicName>
+					<bodyName>imu_link</bodyName>
+					<updateRateHZ>10.0</updateRateHZ>
+					<gaussianNoise>0.0</gaussianNoise>
+					<xyzOffset>0 0 0</xyzOffset>
+					<rpyOffset>0 0 0</rpyOffset>
+					<frameName>imu_link</frameName>
+					<initialOrientationAsReference>false</initialOrientationAsReference>
+				</plugin>
+				<pose>0 0 0 0 0 0</pose>
+			</sensor>
+		</gazebo>
 	</macro>
 	<!-- END IMU macro -->

File: soma_description/urdf/soma.urdf.xacro (robot description, xacro)
@@ -10,20 +10,20 @@
 	<ackermann_macro parent="base_link" />
 	<!-- Build Velodyne -->
-	<!-- <VLP-16 parent="body_bottom_link" name="velodyne" topic="/velodyne_points">
+	<VLP-16 parent="body_bottom_link" name="velodyne" topic="/velodyne_points">
 		<origin xyz="0.075 0.0 ${1.70 - 0.25}" rpy="0.0 0.0 0.0" />
-	</VLP-16> -->
+	</VLP-16>
 	<!-- Build IMU -->
-	<!-- <imu_macro parent="body_bottom_link">
+	<imu_macro parent="body_bottom_link">
 		<origin xyz="${-0.525 + 0.05/2} 0.0 ${1.40 - 0.25 + 0.025/2}" rpy="0.0 0.0 0.0" />
-	</imu_macro> -->
+	</imu_macro>
 	<!-- Build Realsense -->
 	<!-- Front -->
-	<!-- <realsense_macro parent="body_bottom_link" prefix="f">
+	<realsense_macro parent="body_bottom_link" prefix="f">
 		<origin xyz="0.325 0.0 ${1.10 - 0.25}" rpy="0.0 0.0 0.0" />
-	</realsense_macro> -->
+	</realsense_macro>
 	<!-- Rear -->
-	<!-- <realsense_macro parent="body_bottom_link" prefix="r">
+	<realsense_macro parent="body_bottom_link" prefix="r">
 		<origin xyz="-0.525 0.0 ${1.10 - 0.25}" rpy="0.0 0.0 ${-pi}" />
-	</realsense_macro> -->
+	</realsense_macro>
 	<!-- Gazebo plugins -->
 	<gazebo>

File: soma_description/urdf/virtual_rear_wheel_macro.xacro (robot description, xacro)
@@ -4,6 +4,6 @@
     <macro name="virtual_rear_wheel_macro" params="parent prefix xyz">
         <!-- General properties used for inertia computation -->
-        <property name="mass" value="12" />
-        <property name="radius" value="0.2286" />
+        <property name="mass" value="1" />
+        <property name="radius" value="0.03" />
         <property name="length" value="0.0889" />
         <!-- Joint -->
@@ -13,6 +13,6 @@
             <origin xyz="${xyz}" rpy="${-pi/2} 0 0" />
             <axis xyz="0 0 1" rpy="0 0 0" />
-            <!--limit effort="0.4" velocity="12"/-->
-            <!-- <dynamics damping="0.1"/> -->
+            <limit effort="10" velocity="5"/>
+            <dynamics damping="0.1"/>
         </joint>
         <!-- Transmission -->
@@ -56,8 +56,4 @@
 				Gazebo/Red
             </material>
-            <!-- <mu1 value="2.5" /> -->
-            <!-- <mu2 value="2.5" /> -->
-            <!-- <kp value="1000000" /> -->
-            <!-- <kd value="10" /> -->
         </gazebo>
     </macro>

Commit message: Add sensors to moving base again

File: soma_description/urdf/ackermann_macro.xacro (robot description, xacro)
@@ -130,5 +130,5 @@
 		<gazebo reference="body_top_link">
 			<material>
-						Gazebo/Gray
+				Gazebo/Gray
 			</material>
 		</gazebo>

File: soma_description/urdf/sensors_macro.xacro (robot description, xacro)
@@ -81,3 +81,10 @@
 	</macro>
 	<!-- END Realsense macro -->
+	<!-- Velodyne macro -->
+	<macro name="velodyne_macro" params="parent *origin">
+		<VLP-16 parent="${parent}" name="velodyne" topic="/velodyne_points">
+			<insert_block name="origin" />
+		</VLP-16>
+	</macro>
+	<!-- END Velodyne macro -->
 </robot>

File: soma_description/urdf/soma.urdf.xacro (robot description, xacro)
@@ -9,8 +9,4 @@
 	<!-- Build Ackermann movebase -->
 	<ackermann_macro parent="base_link" />
-	<!-- Build Velodyne -->
-	<VLP-16 parent="body_bottom_link" name="velodyne" topic="/velodyne_points">
-		<origin xyz="0.075 0.0 ${1.70 - 0.25}" rpy="0.0 0.0 0.0" />
-	</VLP-16>
 	<!-- Build IMU -->
 	<imu_macro parent="body_bottom_link">
@@ -26,4 +22,8 @@
 		<origin xyz="-0.525 0.0 ${1.10 - 0.25}" rpy="0.0 0.0 ${-pi}" />
 	</realsense_macro>
+	<!-- Build Velodyne -->
+	<velodyne_macro parent="body_bottom_link">
+		<origin xyz="0.075 0.0 ${1.70 - 0.25}" rpy="0.0 0.0 0.0" />
+	</velodyne_macro>
 	<!-- Gazebo plugins -->
 	<gazebo>
@@ -31,7 +31,8 @@
    		implementation of the hardware_interface::RobotHW -->
 		<plugin name="gazebo_ros_control" filename="libgazebo_ros_control.so">
-			<robotNamespace>/soma</robotNamespace>
+			<robotNamespace>/</robotNamespace>
 			<robotSimType>steer_bot_hardware_gazebo/SteerBotHardwareGazebo</robotSimType>
-			<legacyModeNS>false</legacyModeNS>
+			<!-- <robotSimType>gazebo_ros_control/DefaultRobotHWSim</robotSimType> -->
+			<legacyModeNS>true</legacyModeNS>
 		</plugin>
 	</gazebo>
