Commit message: fix urdf for noetic

File: soma_description/urdf/ackermann_macro.xacro (robot description, xacro)
@@ -4,16 +4,16 @@
 <robot xmlns:xacro="http://www.ros.org/wiki/xacro" name="soma">
 	<!-- Include files -->
-	<include filename="$(find soma_description)/urdf/utils.xacro" />
-	<include filename="$(find soma_description)/urdf/front_steer_macro.xacro" />
-	<include filename="$(find soma_description)/urdf/front_wheel_macro.xacro" />
-	<include filename="$(find soma_description)/urdf/rear_wheel_macro.xacro" />
-	<include filename="$(find soma_description)/urdf/virtual_rear_wheel_macro.xacro" />
+	<xacro:include filename="$(find soma_description)/urdf/utils.xacro" />
+	<xacro:include filename="$(find soma_description)/urdf/front_steer_macro.xacro" />
+	<xacro:include filename="$(find soma_description)/urdf/front_wheel_macro.xacro" />
+	<xacro:include filename="$(find soma_description)/urdf/rear_wheel_macro.xacro" />
+	<xacro:include filename="$(find soma_description)/urdf/virtual_rear_wheel_macro.xacro" />
 	<!-- Ackermann macro -->
-	<macro name="ackermann_macro" params="parent">
+	<xacro:macro name="ackermann_macro" params="parent">
 		<!-- General properties used for inertia computation -->
-		<property name="mass" value="250" />
-		<property name="width" value="1.05" />
-		<property name="depth" value="0.70" />
-		<property name="height" value="1.7" />
+		<xacro:property name="mass" value="250" />
+		<xacro:property name="width" value="1.05" />
+		<xacro:property name="depth" value="0.70" />
+		<xacro:property name="height" value="1.7" />
 		<!-- Bottom body joint -->
 		<joint name="body_bottom_joint" type="fixed">
@@ -29,5 +29,5 @@
 				<mass value="${0.8*mass}" />
 				<!-- Inertia matrix of a parallelepiped -->
-				<parallelepiped_inertia mass="${0.8*mass}" width="${width}" height="0.5" depth="${depth}" />
+				<xacro:parallelepiped_inertia mass="${0.8*mass}" width="${width}" height="0.5" depth="${depth}" />
 				<!-- Old values: ixx = iyy = izz = 0.001 -->
 			</inertial>
@@ -68,5 +68,5 @@
 				<mass value="${0.19*mass}" />
 				<!-- Inertia matrix of a parallelepiped -->
-				<parallelepiped_inertia mass="${0.19*mass}" width="0.85" height="0.9" depth="${depth}" />
+				<xacro:parallelepiped_inertia mass="${0.19*mass}" width="0.85" height="0.9" depth="${depth}" />
 				<!-- Old values: ixx = iyy = izz = 0.001 -->
 			</inertial>
@@ -107,5 +107,5 @@
 				<mass value="${0.01*mass}" />
 				<!-- Inertia matrix of a parallelepiped -->
-				<parallelepiped_inertia mass="${0.01*mass}" width="0.05" height="0.3" depth="0.05" />
+				<xacro:parallelepiped_inertia mass="${0.01*mass}" width="0.05" height="0.3" depth="0.05" />
 				<!-- Old values: ixx = iyy = izz = 0.001 -->
 			</inertial>
@@ -134,11 +134,11 @@
 		</gazebo>
 		<!-- Build links and joints for ackermann_steering_controller -->
-		<front_steer_macro parent="body_bottom_link" prefix="ackermann" xyz="${width/2} 0 ${-0.5/2}" />
-		<virtual_rear_wheel_macro parent="body_bottom_link" prefix="ackermann" xyz="${-width/2} 0 ${-0.5/2}" />
+		<xacro:front_steer_macro parent="body_bottom_link" prefix="ackermann" xyz="${width/2} 0 ${-0.5/2}" />
+		<xacro:virtual_rear_wheel_macro parent="body_bottom_link" prefix="ackermann" xyz="${-width/2} 0 ${-0.5/2}" />
 		<!-- Build wheels -->
-		<front_wheel_macro parent="body_bottom_link" prefix="left" xyz="${width/2} ${depth/2 + 0.0889} ${-0.5/2}" />
-		<front_wheel_macro parent="body_bottom_link" prefix="right" xyz="${width/2} ${-depth/2 - 0.0889} ${-0.5/2}" />
-		<rear_wheel_macro parent="body_bottom_link" prefix="left" xyz="${-width/2} ${depth/2 + 0.0889} ${-0.5/2}" />
-		<rear_wheel_macro parent="body_bottom_link" prefix="right" xyz="${-width/2} ${-depth/2 - 0.0889} ${-0.5/2}" />
-	</macro>
+		<xacro:front_wheel_macro parent="body_bottom_link" prefix="left" xyz="${width/2} ${depth/2 + 0.0889} ${-0.5/2}" />
+		<xacro:front_wheel_macro parent="body_bottom_link" prefix="right" xyz="${width/2} ${-depth/2 - 0.0889} ${-0.5/2}" />
+		<xacro:rear_wheel_macro parent="body_bottom_link" prefix="left" xyz="${-width/2} ${depth/2 + 0.0889} ${-0.5/2}" />
+		<xacro:rear_wheel_macro parent="body_bottom_link" prefix="right" xyz="${-width/2} ${-depth/2 - 0.0889} ${-0.5/2}" />
+	</xacro:macro>
 </robot>

File: soma_description/urdf/front_steer_macro.xacro (robot description, xacro)
@@ -2,5 +2,5 @@
 <robot xmlns:xacro="http://www.ros.org/wiki/xacro" name="soma">
     <!-- Front wheel macro -->
-    <macro name="front_steer_macro" params="parent prefix xyz">
+    <xacro:macro name="front_steer_macro" params="parent prefix xyz">
         <!-- General properties used for inertia computation -->
         <!-- Joints -->
@@ -47,5 +47,5 @@
                 <origin xyz="0 0 0.3" rpy="0 0 0" />
                 <mass value="0.2"/>
-                <cylinder_inertia mass="0.2" radius="0.1" height="0.05"/>
+                <xacro:cylinder_inertia mass="0.2" radius="0.1" height="0.05"/>
             </inertial>
         </link>
@@ -59,5 +59,5 @@
             <provideFeedback>true</provideFeedback>
         </gazebo> -->
-    </macro>
+    </xacro:macro>
     <!-- END front wheel macro -->
 </robot>

File: soma_description/urdf/front_wheel_macro.xacro (robot description, xacro)
@@ -2,9 +2,9 @@
 <robot xmlns:xacro="http://www.ros.org/wiki/xacro" name="soma">
     <!-- Front wheel macro -->
-    <macro name="front_wheel_macro" params="parent prefix xyz">
+    <xacro:macro name="front_wheel_macro" params="parent prefix xyz">
         <!-- General properties used for inertia computation -->
-        <property name="mass" value="12" />
-        <property name="radius" value="0.2286" />
-        <property name="length" value="0.0889" />
+        <xacro:property name="mass" value="12" />
+        <xacro:property name="radius" value="0.2286" />
+        <xacro:property name="length" value="0.0889" />
         <!-- Joints -->
         <joint name="${prefix}_front_wheel_hinge" type="revolute">
@@ -68,5 +68,5 @@
                 <origin xyz="0 0 0" rpy="0 0 0" />
                 <mass value="${mass}"/>
-                <cylinder_inertia mass="${mass}" radius="${radius}" height="${length}" />
+                <xacro:cylinder_inertia mass="${mass}" radius="${radius}" height="${length}" />
             </inertial>
         </link>
@@ -91,5 +91,5 @@
                 <origin xyz="0 0 0.3" rpy="0 0 0" />
                 <mass value="0.2"/>
-                <cylinder_inertia mass="0.2" radius="0.07" height="0.05"/>
+                <xacro:cylinder_inertia mass="0.2" radius="0.07" height="0.05"/>
             </inertial>
         </link>
@@ -113,5 +113,5 @@
             <!-- <kd value="10" /> -->
         </gazebo>
-    </macro>
+    </xacro:macro>
     <!-- END front wheel macro -->
 </robot>

File: soma_description/urdf/rear_wheel_macro.xacro (robot description, xacro)
@@ -2,9 +2,9 @@
 <robot xmlns:xacro="http://www.ros.org/wiki/xacro" name="soma">
     <!-- Rear wheel macro -->
-    <macro name="rear_wheel_macro" params="parent prefix xyz">
+    <xacro:macro name="rear_wheel_macro" params="parent prefix xyz">
         <!-- General properties used for inertia computation -->
-        <property name="mass" value="12" />
-        <property name="radius" value="0.2286" />
-        <property name="length" value="0.0889" />
+        <xacro:property name="mass" value="12" />
+        <xacro:property name="radius" value="0.2286" />
+        <xacro:property name="length" value="0.0889" />
         <!-- Joint -->
         <joint name="${prefix}_rear_wheel_rotate" type="continuous">
@@ -48,5 +48,5 @@
                 <origin xyz="0 0 0" rpy="0 0 0" />
                 <mass value="${mass}"/>
-                <cylinder_inertia mass="${mass}" radius="${radius}" height="${length}" />
+                <xacro:cylinder_inertia mass="${mass}" radius="${radius}" height="${length}" />
             </inertial>
         </link>
@@ -61,5 +61,5 @@
             <!-- <kd value="10" /> -->
         </gazebo>
-    </macro>
+    </xacro:macro>
     <!-- END rear wheel macro -->
 </robot>

File: soma_description/urdf/sensors_macro.xacro (robot description, xacro)
@@ -1,22 +1,22 @@
 <?xml version="1.0"?>
 <robot xmlns:xacro="http://www.ros.org/wiki/xacro" name="soma">
-	<property name="camera_enabled" value="false"/>
-	<property name="lidar_enabled" value="true"/>
-	<property name="imu_enabled" value="false"/>
+	<xacro:property name="camera_enabled" value="true"/>
+	<xacro:property name="lidar_enabled" value="true"/>
+	<xacro:property name="imu_enabled" value="false"/>
 	<!-- Include files -->
 	<if value="${camera_enabled}">
-		<include filename="$(find realsense2_description)/urdf/_d435.urdf.xacro" />
+		<xacro:include filename="$(find realsense2_description)/urdf/_d435.urdf.xacro" />
 	</if>
 	<if value="${lidar_enabled}">
-		<include filename="$(find velodyne_description)/urdf/VLP-16.urdf.xacro" />
+		<xacro:include filename="$(find velodyne_description)/urdf/VLP-16.urdf.xacro" />
 	</if>
 	<!-- IMU macro -->
 	<if value="${imu_enabled}">
-		<macro name="imu_macro" params="parent *origin">
+		<xacro:macro name="imu_macro" params="parent *origin">
 			<!-- General properties used for inertia computation -->
-			<property name="mass" value="0.2" />
-			<property name="width" value="0.05" />
-			<property name="depth" value="0.05" />
-			<property name="height" value="0.025" />
+			<xacro:property name="mass" value="0.2" />
+			<xacro:property name="width" value="0.05" />
+			<xacro:property name="depth" value="0.05" />
+			<xacro:property name="height" value="0.025" />
 			<!-- Joint -->
 			<joint name="imu_joint" type="fixed">
@@ -75,10 +75,10 @@
 				</sensor>
 			</gazebo>
-		</macro>
+		</xacro:macro>
 	</if>
 	<!-- END IMU macro -->
 	<!-- Realsense macro -->
 	<if value="${camera_enabled}">
-		<macro name="realsense_macro" params="parent prefix *origin">
+		<xacro:macro name="realsense_macro" params="parent prefix *origin">
 			<link name="camera_${prefix}_mount_link" />
 			<joint name="camera_${prefix}_mount_joint" type="fixed">
@@ -90,15 +90,15 @@
 				<origin xyz="0.0 0.0 0.0" rpy="0.0 0.2617 0.0" />
 			</sensor_d435>
-		</macro>
+		</xacro:macro>
 	</if>
 	<!-- END Realsense macro -->
 	<!-- Velodyne macro -->
 	<if value="${lidar_enabled}">
-		<macro name="velodyne_macro" params="parent *origin">
+		<xacro:macro name="velodyne_macro" params="parent *origin">
 			<VLP-16 parent="${parent}" name="velodyne" topic="/velodyne_points" min_range="0.0" max_range="5.0" noise="0.0">
 				<!-- <VLP-16 parent="${parent}" name="velodyne" topic="/velodyne_points" min_range="0.9" max_range="130.0" noise="0.008"> -->
 				<insert_block name="origin" />
 			</VLP-16>
-		</macro>
+		</xacro:macro>
 	</if>
 	<!-- END Velodyne macro -->

File: soma_description/urdf/soma.urdf.xacro (robot description, xacro)
@@ -1,41 +1,41 @@
 <?xml version="1.0"?>
 <robot xmlns:xacro="http://www.ros.org/wiki/xacro" name="soma">
-	<property name="sensors_enabled" value="true"/>
+	<xacro:property name="sensors_enabled" value="true"/>
 	<!-- Include files -->
-	<include filename="$(find soma_description)/urdf/ackermann_macro.xacro" />
-	<if value="${sensors_enabled}">
-		<include filename="$(find soma_description)/urdf/sensors_macro.xacro" />
-	</if>
+	<xacro:include filename="$(find soma_description)/urdf/ackermann_macro.xacro" />
+	<xacro:if value="${sensors_enabled}">
+		<xacro:include filename="$(find soma_description)/urdf/sensors_macro.xacro" />
+	</xacro:if>
 	<!-- Empty link to use Gazebo -->
 	<link name="base_link" />
 	<!-- Build Ackermann movebase -->
-	<ackermann_macro parent="base_link" />
-	<if value="${sensors_enabled}">
+	<xacro:ackermann_macro parent="base_link" />
+	<xacro:if value="${sensors_enabled}">
 		<!-- Build IMU -->
-		<if value="${imu_enabled}">
-			<imu_macro parent="body_bottom_link">
+		<xacro:if value="${imu_enabled}">
+			<xacro:imu_macro parent="body_bottom_link">
 				<origin xyz="${-0.525 + 0.05/2} 0.0 ${1.40 - 0.25 + 0.025/2}" rpy="0.0 0.0 0.0" />
-			</imu_macro>
-		</if>
+			</xacro:imu_macro>
+		</xacro:if>
 		<!-- Build Realsense -->
 		<!-- Front -->
-		<if value="${camera_enabled}">
-			<realsense_macro parent="body_bottom_link" prefix="f">
+		<xacro:if value="${camera_enabled}">
+			<xacro:realsense_macro parent="body_bottom_link" prefix="f">
 				<origin xyz="0.325 0.0 ${1.10 - 0.25}" rpy="0.0 0.0 0.0" />
-			</realsense_macro>
-		</if>
+			</xacro:realsense_macro>
+		</xacro:if>
 		<!-- Rear -->
-		<if value="${camera_enabled}">
-			<realsense_macro parent="body_bottom_link" prefix="r">
+		<xacro:if value="${camera_enabled}">
+			<xacro:realsense_macro parent="body_bottom_link" prefix="r">
 				<origin xyz="-0.525 0.0 ${1.10 - 0.25}" rpy="0.0 0.0 ${-pi}" />
-			</realsense_macro>
-		</if>
+			</xacro:realsense_macro>
+		</xacro:if>
 		<!-- Build Velodyne -->
-		<if value="${lidar_enabled}">
-			<velodyne_macro parent="body_bottom_link">
+		<xacro:if value="${lidar_enabled}">
+			<xacro:velodyne_macro parent="body_bottom_link">
 				<origin xyz="0.075 0.0 ${1.70 - 0.25}" rpy="0.0 0.0 0.0" />
-			</velodyne_macro>
-		</if>
-	</if>
+			</xacro:velodyne_macro>
+		</xacro:if>
+	</xacro:if>
 	<!-- Gazebo plugins -->
 	<gazebo>

File: soma_description/urdf/utils.xacro (robot description, xacro)
@@ -3,20 +3,20 @@
     <!-- Materials -->
 	<material name="gray">
-		<color rgba="0.5 0.5 0.5 2.5" />
+		<color rgba="0.5 0.5 0.5" />
 	</material>
 	<material name="red">
-		<color rgba="1.0 0.0 0.0 2.5" />
+		<color rgba="1.0 0.0 0.0" />
 	</material>
     <!-- Cylinder inertia -->
-    <macro name="cylinder_inertia" params="mass radius height">
+    <xacro:macro name="cylinder_inertia" params="mass radius height">
         <inertia ixx="${mass / 12 * (3 * radius ** 2 + height ** 2)}" ixy="0.0"
 				 ixz="0.0" iyy="${mass / 12 * (3 * radius ** 2 + height ** 2)}"
 				 iyz="0.0" izz="${mass / 2 * radius ** 2}" />
-    </macro>
+    </xacro:macro>
     <!-- Parallelepiped inertia -->
-    <macro name="parallelepiped_inertia" params="mass width height depth">
+    <xacro:macro name="parallelepiped_inertia" params="mass width height depth">
         <inertia ixx="${mass / 12 * (depth ** 2 + height ** 2)}" ixy="0.0"
 				 ixz="0.0" iyy="${mass / 12 * (width ** 2 + height ** 2)}"
 				 iyz="0.0" izz="${mass / 12 * (width ** 2 + depth ** 2)}" />
-    </macro>
+    </xacro:macro>
 </robot>

File: soma_description/urdf/virtual_rear_wheel_macro.xacro (robot description, xacro)
@@ -2,9 +2,9 @@
 <robot xmlns:xacro="http://www.ros.org/wiki/xacro" name="soma">
     <!-- Rear wheel macro -->
-    <macro name="virtual_rear_wheel_macro" params="parent prefix xyz">
+    <xacro:macro name="virtual_rear_wheel_macro" params="parent prefix xyz">
         <!-- General properties used for inertia computation -->
-        <property name="mass" value="12" />
-        <property name="radius" value="0.03" />
-        <property name="length" value="0.0889" />
+        <xacro:property name="mass" value="12" />
+        <xacro:property name="radius" value="0.03" />
+        <xacro:property name="length" value="0.0889" />
         <!-- Joint -->
         <joint name="${prefix}_virtual_rear_wheel_rotate" type="continuous">
@@ -48,5 +48,5 @@
                 <origin xyz="0 0 0" rpy="0 0 0" />
                 <mass value="${mass}"/>
-                <cylinder_inertia mass="${mass}" radius="${radius}" height="${length}" />
+                <xacro:cylinder_inertia mass="${mass}" radius="${radius}" height="${length}" />
             </inertial>
         </link>
@@ -57,5 +57,5 @@
             </material>
         </gazebo>
-    </macro>
+    </xacro:macro>
     <!-- END rear wheel macro -->
 </robot>

Commit message: Fix gazebo simulation error

File: soma_description/urdf/ackermann_macro.xacro (robot description, xacro)
@@ -12,5 +12,6 @@
 	<xacro:macro name="ackermann_macro" params="parent">
 		<!-- General properties used for inertia computation -->
-		<xacro:property name="mass" value="250" />
+		<!-- <xacro:property name="mass" value="250" /> -->
+		<xacro:property name="mass" value="10" />
 		<xacro:property name="width" value="1.05" />
 		<xacro:property name="depth" value="0.70" />
@@ -44,5 +45,5 @@
 				<origin xyz="0.0 0.0 0.0" rpy="0.0 0.0 0.0" />
 				<geometry>
-					<box size="${width} ${depth} 0.5" />
+					<box size="${width}-0.2 ${depth}-0.1 0.5" />
 				</geometry>
 			</collision>
@@ -83,5 +84,5 @@
 				<origin xyz="0.0 0.0 0.0" rpy="0.0 0.0 0.0" />
 				<geometry>
-					<box size="0.85 ${depth} 0.9" />
+					<box size="0.75 ${depth} 0.9" />
 				</geometry>
 			</collision>

File: soma_description/urdf/intel_realsense.urdf.xacro (robot description, xacro)
@@ -82,4 +82,10 @@
         <material name="white" />
       </visual>
+      <inertial>
+        <!-- The following are not reliable values, and should not be used for modeling -->
+        <mass value="0.564" />
+        <origin xyz="0.0115 0 0.0100" />
+        <inertia ixx="0.003881243" ixy="0.0" ixz="0.0" iyy="0.000498940" iyz="0.0" izz="0.003879257" />
+      </inertial>
     </link>
     <joint type="fixed" name="${prefix}_realsense_lens_joint">

Commit message: Move base_link to the middle of rear axis

File: soma_description/urdf/ackermann_macro.xacro (robot description, xacro)
@@ -20,5 +20,5 @@
 			<parent link="${parent}" />
 			<child link="body_bottom_link" />
-			<origin xyz="0 0 ${0.2286 + 0.5/2}" rpy="0.0 0.0 0.0" />
+			<origin xyz="${0.5*width} 0 ${0.2286 + 0.5/2}" rpy="0.0 0.0 0.0" />
 		</joint>
 		<!-- Bottom body link -->
@@ -59,5 +59,5 @@
 			<parent link="${parent}" />
 			<child link="body_middle_link" />
-			<origin xyz="-0.1 0 ${0.2286 + 0.5 + 0.9/2}" rpy="0.0 0.0 0.0" />
+			<origin xyz="${0.5*width - 0.1} 0 ${0.2286 + 0.5 + 0.9/2}" rpy="0.0 0.0 0.0" />
 		</joint>
 		<!-- Middle body link -->
@@ -98,5 +98,5 @@
 			<parent link="${parent}" />
 			<child link="body_top_link" />
-			<origin xyz="0.075 0 ${0.2286 + 0.5 + 0.9 + 0.3/2}" rpy="0.0 0.0 0.0" />
+			<origin xyz="${0.5*width + 0.075} 0 ${0.2286 + 0.5 + 0.9 + 0.3/2}" rpy="0.0 0.0 0.0" />
 		</joint>
 		<!-- Top body link -->
